File: hardware/cpld-cpu.kicad_pcb (KiCad board)
At the start: 2 copper layers, 0 parts

Commit message: Most of the schematic done (just missing RAM/mmappedio)
Parts:
- added C1: 100n, Capacitors_SMD:C_0805_HandSoldering, F.Cu at (214.9, 136.8)
- added C10: 100n, Capacitors_SMD:C_0805_HandSoldering, F.Cu at (224.2, 133.0)
- added C11: 100n, Capacitors_SMD:C_0805_HandSoldering, F.Cu at (228.1, 128.9)
- added C12: 100n, Capacitors_SMD:C_0805_HandSoldering, F.Cu at (209.9, 147.9)
- added C13: 100n, Capacitors_SMD:C_0805_HandSoldering, F.Cu at (232.9, 125.2)
- added C14: 100n, Capacitors_SMD:C_0805_HandSoldering, F.Cu at (200.5, 153.9)
- added C15: 100n, Capacitors_SMD:C_0805_HandSoldering, F.Cu at (228.3, 127.0)
- added C16: 100n, Capacitors_SMD:C_0805_HandSoldering, F.Cu at (219.6, 134.8)
- added C17: 100n, Capacitors_SMD:C_0805_HandSoldering, F.Cu at (195.7, 157.7)
- added C18: 100n, Capacitors_SMD:C_0805_HandSoldering, F.Cu at (214.9, 138.6)
- added C19: 100n, Capacitors_SMD:C_0805_HandSoldering, F.Cu at (228.3, 125.2)
- added C2: 100n, Capacitors_SMD:C_0805_HandSoldering, F.Cu at (223.4, 131.2)
- added C20: 100n, Capacitors_SMD:C_0805_HandSoldering, F.Cu at (205.4, 147.9)
- added C21: 100n, Capacitors_SMD:C_0805_HandSoldering, F.Cu at (223.6, 129.3)
- added C22: 100n, Capacitors_SMD:C_0805_HandSoldering, F.Cu at (219.6, 133.0)
- added C23: 100n, Capacitors_SMD:C_0805_HandSoldering, F.Cu at (210.1, 142.5)
- added C24: 100n, Capacitors_SMD:C_0805_HandSoldering, F.Cu at (218.8, 131.2)
- added C25: 100n, Capacitors_SMD:C_0805_HandSoldering, F.Cu at (228.3, 123.4)
- added C26: 100n, Capacitors_SMD:C_0805_HandSoldering, F.Cu at (205.0, 151.6)
- added C27: 100n, Capacitors_SMD:C_0805_HandSoldering, F.Cu at (195.7, 155.9)
- added C28: 100n, Capacitors_SMD:C_0805_HandSoldering, F.Cu at (223.6, 127.4)
- added C29: 100n, Capacitors_SMD:C_0805_HandSoldering, F.Cu at (200.5, 150.3)
- added C3: 100n, Capacitors_SMD:C_0805_HandSoldering, F.Cu at (214.9, 140.5)
- added C30: 100n, Capacitors_SMD:C_0805_HandSoldering, F.Cu at (205.4, 146.1)
- added C31: 100n, Capacitors_SMD:C_0805_HandSoldering, F.Cu at (232.9, 123.4)
- added C32: 100n, Capacitors_SMD:C_0805_HandSoldering, F.Cu at (200.5, 152.1)
- added C33: 100n, Capacitors_SMD:C_0805_HandSoldering, F.Cu at (219.4, 138.6)
- added C4: 100n, Capacitors_SMD:C_0805_HandSoldering, F.Cu at (205.4, 149.8)
- added C5: 100n, Capacitors_SMD:C_0805_HandSoldering, F.Cu at (209.9, 146.1)
- added C6: 100n, Capacitors_SMD:C_0805_HandSoldering, F.Cu at (200.3, 155.9)
- added C7: 100n, Capacitors_SMD:C_0805_HandSoldering, F.Cu at (219.4, 136.8)
- added C8: 100n, Capacitors_SMD:C_0805_HandSoldering, F.Cu at (210.1, 144.3)
- added C9: 100n, Capacitors_SMD:C_0805_HandSoldering, F.Cu at (214.7, 142.5)
- added D1: LED_Small, LEDs:LED_0805_HandSoldering, F.Cu at (167.3, 150.9)
- added D10: LED_Small, LEDs:LED_0805_HandSoldering, F.Cu at (143.6, 153.5)
- added D11: LED_Small, LEDs:LED_0805_HandSoldering, F.Cu at (148.3, 150.9)
- added D12: LED_Small, LEDs:LED_0805_HandSoldering, F.Cu at (153.1, 149.1)
- added D13: LED_Small, LEDs:LED_0805_HandSoldering, F.Cu at (157.8, 149.1)
- added D14: LED_Small, LEDs:LED_0805_HandSoldering, F.Cu at (153.1, 150.9)
- added D15: LED_Small, LEDs:LED_0805_HandSoldering, F.Cu at (148.3, 152.8)
- added D16: LED_Small, LEDs:LED_0805_HandSoldering, F.Cu at (153.1, 152.8)
- added D17: LED_Small, LEDs:LED_0805_HandSoldering, F.Cu at (143.6, 149.8)
- added D18: LED_Small, LEDs:LED_0805_HandSoldering, F.Cu at (176.8, 154.6)
- added D19: LED_Small, LEDs:LED_0805_HandSoldering, F.Cu at (209.4, 125.5)
- added D2: LED_Small, LEDs:LED_0805_HandSoldering, F.Cu at (167.3, 152.8)
- added D20: LED_Small, LEDs:LED_0805_HandSoldering, F.Cu at (204.7, 131.1)
- added D21: LED_Small, LEDs:LED_0805_HandSoldering, F.Cu at (176.8, 158.3)
- added D22: LED_Small, LEDs:LED_0805_HandSoldering, F.Cu at (167.3, 158.3)
- added D23: LED_Small, LEDs:LED_0805_HandSoldering, F.Cu at (162.6, 156.5)
- added D24: LED_Small, LEDs:LED_0805_HandSoldering, F.Cu at (157.8, 158.4)
- added D25: LED_Small, LEDs:LED_0805_HandSoldering, F.Cu at (162.6, 158.4)
- added D26: LED_Small, LEDs:LED_0805_HandSoldering, F.Cu at (191.2, 135.3)
- added D27: LED_Small, LEDs:LED_0805_HandSoldering, F.Cu at (167.3, 154.6)
- added D28: LED_Small, LEDs:LED_0805_HandSoldering, F.Cu at (167.3, 156.5)
- added D29: LED_Small, LEDs:LED_0805_HandSoldering, F.Cu at (172.1, 150.9)
- added D3: LED_Small, LEDs:LED_0805_HandSoldering, F.Cu at (162.6, 152.8)
- added D30: LED_Small, LEDs:LED_0805_HandSoldering, F.Cu at (176.8, 149.1)
- added D31: LED_Small, LEDs:LED_0805_HandSoldering, F.Cu at (214.2, 121.8)
- added D32: LED_Small, LEDs:LED_0805_HandSoldering, F.Cu at (172.1, 152.8)
- added D33: LED_Small, LEDs:LED_0805_HandSoldering, F.Cu at (157.8, 156.5)
- added D34: LED_Small, LEDs:LED_0805_HandSoldering, F.Cu at (204.7, 121.8)
- added D35: LED_Small, LEDs:LED_0805_HandSoldering, F.Cu at (209.4, 121.8)
- added D36: LED_Small, LEDs:LED_0805_HandSoldering, F.Cu at (204.7, 123.7)
- added D37: LED_Small, LEDs:LED_0805_HandSoldering, F.Cu at (204.7, 125.5)
- added D38: LED_Small, LEDs:LED_0805_HandSoldering, F.Cu at (172.1, 154.6)
- added D39: LED_Small, LEDs:LED_0805_HandSoldering, F.Cu at (172.1, 156.5)
- added D4: LED_Small, LEDs:LED_0805_HandSoldering, F.Cu at (162.6, 154.7)
- added D40: LED_Small, LEDs:LED_0805_HandSoldering, F.Cu at (172.1, 158.3)
- added D41: LED_Small, LEDs:LED_0805_HandSoldering, F.Cu at (176.8, 150.9)
- added D42: LED_Small, LEDs:LED_0805_HandSoldering, F.Cu at (176.8, 152.8)
- added D43: LED_Small, LEDs:LED_0805_HandSoldering, F.Cu at (181.6, 148.7)
- added D44: LED_Small, LEDs:LED_0805_HandSoldering, F.Cu at (196.0, 135.3)
- added D45: LED_Small, LEDs:LED_0805_HandSoldering, F.Cu at (191.2, 137.1)
- added D46: LED_Small, LEDs:LED_0805_HandSoldering, F.Cu at (191.2, 139.0)
- added D47: LED_Small, LEDs:LED_0805_HandSoldering, F.Cu at (148.3, 154.6)
- added D48: LED_Small, LEDs:LED_0805_HandSoldering, F.Cu at (191.2, 140.8)
- added D49: LED_Small, LEDs:LED_0805_HandSoldering, F.Cu at (196.0, 137.1)
- added D5: LED_Small, LEDs:LED_0805_HandSoldering, F.Cu at (157.8, 154.7)
- added D50: LED_Small, LEDs:LED_0805_HandSoldering, F.Cu at (181.6, 150.6)
- added D51: LED_Small, LEDs:LED_0805_HandSoldering, F.Cu at (181.6, 152.4)
- added D52: LED_Small, LEDs:LED_0805_HandSoldering, F.Cu at (191.2, 142.7)
- added D6: LED_Small, LEDs:LED_0805_HandSoldering, F.Cu at (172.1, 149.1)
- added D7: LED_Small, LEDs:LED_0805_HandSoldering, F.Cu at (143.6, 155.3)
- added D8: LED_Small, LEDs:LED_0805_HandSoldering, F.Cu at (148.3, 149.1)
- added D9: LED_Small, LEDs:LED_0805_HandSoldering, F.Cu at (143.6, 151.6)
- added J1: Acc, Pin_Headers:Pin_Header_Straight_1x05_Pitch2.54mm, F.Cu at (161.3, 109.3)
- added J10: PC_H, Pin_Headers:Pin_Header_Straight_1x05_Pitch2.54mm, F.Cu at (150.3, 109.3)
- added J11: Conn_01x05, Pin_Headers:Pin_Header_Straight_1x05_Pitch2.54mm, F.Cu at (146.7, 123.1)
- added J2: X, Pin_Headers:Pin_Header_Straight_1x05_Pitch2.54mm, F.Cu at (164.9, 109.3)
- added J3: IR, Pin_Headers:Pin_Header_Straight_1x05_Pitch2.54mm, F.Cu at (168.6, 109.3)
- added J4: AXM, Pin_Headers:Pin_Header_Straight_1x05_Pitch2.54mm, F.Cu at (143.0, 123.1)
- added J5: Dec, Pin_Headers:Pin_Header_Straight_1x05_Pitch2.54mm, F.Cu at (157.6, 109.3)
- added J6: AR, Pin_Headers:Pin_Header_Straight_1x05_Pitch2.54mm, F.Cu at (154.0, 109.3)
- added J7: ALU, Pin_Headers:Pin_Header_Straight_1x05_Pitch2.54mm, F.Cu at (143.0, 109.3)
- added J8: PC_L, Pin_Headers:Pin_Header_Straight_1x05_Pitch2.54mm, F.Cu at (146.7, 109.3)
- added J9: Conn_01x05, Pin_Headers:Pin_Header_Straight_1x05_Pitch2.54mm, F.Cu at (143.0, 136.9)
- added R1: 2k, Resistors_SMD:R_0805_HandSoldering, F.Cu at (176.8, 156.5)
- added R10: 2k, Resistors_SMD:R_0805_HandSoldering, F.Cu at (231.3, 108.4)
- added R11: 2k, Resistors_SMD:R_0805_HandSoldering, F.Cu at (226.6, 112.1)
- added R12: 2k, Resistors_SMD:R_0805_HandSoldering, F.Cu at (200.7, 137.2)
- added R13: 2k, Resistors_SMD:R_0805_HandSoldering, F.Cu at (186.3, 150.6)
- added R14: 2k, Resistors_SMD:R_0805_HandSoldering, F.Cu at (196.0, 140.9)
- added R15: 2k, Resistors_SMD:R_0805_HandSoldering, F.Cu at (181.6, 156.2)
- added R16: 2k, Resistors_SMD:R_0805_HandSoldering, F.Cu at (191.2, 146.4)
- added R17: 2k, Resistors_SMD:R_0805_HandSoldering, F.Cu at (191.2, 144.5)
- added R18: 2k, Resistors_SMD:R_0805_HandSoldering, F.Cu at (181.6, 154.3)
- added R19: 2k, Resistors_SMD:R_0805_HandSoldering, F.Cu at (214.2, 123.7)
- added R2: 2k, Resistors_SMD:R_0805_HandSoldering, F.Cu at (204.7, 127.4)
- added R20: 2k, Resistors_SMD:R_0805_HandSoldering, F.Cu at (209.4, 129.3)
- added R21: 2k, Resistors_SMD:R_0805_HandSoldering, F.Cu at (196.0, 142.7)
- added R22: 2k, Resistors_SMD:R_0805_HandSoldering, F.Cu at (218.9, 121.8)
- added R23: 2k, Resistors_SMD:R_0805_HandSoldering, F.Cu at (196.0, 144.6)
- added R24: 2k, Resistors_SMD:R_0805_HandSoldering, F.Cu at (209.4, 131.2)
- added R25: 2k, Resistors_SMD:R_0805_HandSoldering, F.Cu at (214.2, 125.6)
- added R26: 470, Resistors_SMD:R_0805_HandSoldering, F.Cu at (191.2, 148.3)
- added R27: 470, Resistors_SMD:R_0805_HandSoldering, F.Cu at (181.6, 158.0)
- added R28: 470, Resistors_SMD:R_0805_HandSoldering, F.Cu at (186.3, 152.5)
- added R29: 470, Resistors_SMD:R_0805_HandSoldering, F.Cu at (231.3, 119.7)
- added R3: 2k, Resistors_SMD:R_0805_HandSoldering, F.Cu at (204.7, 129.3)
- added R30: 470, Resistors_SMD:R_0805_HandSoldering, F.Cu at (200.7, 139.0)
- added R31: 470, Resistors_SMD:R_0805_HandSoldering, F.Cu at (226.6, 114.0)
- added R32: 470, Resistors_SMD:R_0805_HandSoldering, F.Cu at (205.5, 134.9)
- added R33: 470, Resistors_SMD:R_0805_HandSoldering, F.Cu at (186.3, 154.4)
- added R34: 470, Resistors_SMD:R_0805_HandSoldering, F.Cu at (231.3, 110.3)
- added R35: 470, Resistors_SMD:R_0805_HandSoldering, F.Cu at (191.1, 150.2)
- added R36: 470, Resistors_SMD:R_0805_HandSoldering, F.Cu at (191.1, 152.1)
- added R37: 470, Resistors_SMD:R_0805_HandSoldering, F.Cu at (231.3, 112.1)
- added R38: 470, Resistors_SMD:R_0805_HandSoldering, F.Cu at (186.3, 156.3)
- added R39: 470, Resistors_SMD:R_0805_HandSoldering, F.Cu at (205.5, 136.8)
- added R4: 2k, Resistors_SMD:R_0805_HandSoldering, F.Cu at (209.4, 123.7)
- added R40: 470, Resistors_SMD:R_0805_HandSoldering, F.Cu at (205.5, 138.6)
- added R41: 470, Resistors_SMD:R_0805_HandSoldering, F.Cu at (226.6, 115.9)
- added R42: 470, Resistors_SMD:R_0805_HandSoldering, F.Cu at (226.6, 117.8)
- added R43: 470, Resistors_SMD:R_0805_HandSoldering, F.Cu at (167.3, 149.1)
- added R44: 470, Resistors_SMD:R_0805_HandSoldering, F.Cu at (200.7, 142.8)
- added R45: 470, Resistors_SMD:R_0805_HandSoldering, F.Cu at (196.0, 146.5)
- added R46: 470, Resistors_SMD:R_0805_HandSoldering, F.Cu at (196.0, 148.4)
- added R47: 2k, Resistors_SMD:R_0805_HandSoldering, F.Cu at (214.2, 127.4)
- added R48: 2k, Resistors_SMD:R_0805_HandSoldering, F.Cu at (214.2, 129.3)
- added R49: 2k, Resistors_SMD:R_0805_HandSoldering, F.Cu at (218.9, 123.7)
- added R5: 2k, Resistors_SMD:R_0805_HandSoldering, F.Cu at (205.5, 144.3)
- added R50: 2k, Resistors_SMD:R_0805_HandSoldering, F.Cu at (223.7, 121.8)
- added R51: 2k, Resistors_SMD:R_0805_HandSoldering, F.Cu at (218.9, 125.6)
- added R52: 2k, Resistors_SMD:R_0805_HandSoldering, F.Cu at (214.2, 131.2)
- added R53: 2k, Resistors_SMD:R_0805_HandSoldering, F.Cu at (200.7, 144.7)
- added R54: 2k, Resistors_SMD:R_0805_HandSoldering, F.Cu at (186.3, 158.1)
- added R55: 2k, Resistors_SMD:R_0805_HandSoldering, F.Cu at (204.7, 133.0)
- added R56: 2k, Resistors_SMD:R_0805_HandSoldering, F.Cu at (209.4, 127.4)
- added R57: 2k, Resistors_SMD:R_0805_HandSoldering, F.Cu at (195.8, 152.1)
- added R58: 470, Resistors_SMD:R_0805_HandSoldering, F.Cu at (215.0, 133.1)
- added R59: 470, Resistors_SMD:R_0805_HandSoldering, F.Cu at (218.9, 129.4)
- added R6: 2k, Resistors_SMD:R_0805_HandSoldering, F.Cu at (196.0, 139.0)
- added R60: 470, Resistors_SMD:R_0805_HandSoldering, F.Cu at (191.1, 157.7)
- added R61: 470, Resistors_SMD:R_0805_HandSoldering, F.Cu at (231.3, 117.8)
- added R62: 470, Resistors_SMD:R_0805_HandSoldering, F.Cu at (210.2, 138.7)
- added R63: 470, Resistors_SMD:R_0805_HandSoldering, F.Cu at (228.4, 121.5)
- added R64: 470, Resistors_SMD:R_0805_HandSoldering, F.Cu at (215.0, 135.0)
- added R65: 470, Resistors_SMD:R_0805_HandSoldering, F.Cu at (195.8, 154.0)
- added R66: 2k, Resistors_SMD:R_0805_HandSoldering, F.Cu at (223.7, 125.6)
- added R67: 2k, Resistors_SMD:R_0805_HandSoldering, F.Cu at (200.7, 148.4)
- added R68: 2k, Resistors_SMD:R_0805_HandSoldering, F.Cu at (200.7, 140.9)
- added R69: 2k, Resistors_SMD:R_0805_HandSoldering, F.Cu at (231.3, 114.0)
- added R7: 2k, Resistors_SMD:R_0805_HandSoldering, F.Cu at (186.3, 148.7)
- added R70: 2k, Resistors_SMD:R_0805_HandSoldering, F.Cu at (148.3, 156.5)
- added R71: 2k, Resistors_SMD:R_0805_HandSoldering, F.Cu at (143.6, 158.4)
- added R72: 2k, Resistors_SMD:R_0805_HandSoldering, F.Cu at (148.3, 158.4)
- added R73: 2k, Resistors_SMD:R_0805_HandSoldering, F.Cu at (162.6, 149.1)
- added R74: 470, Resistors_SMD:R_0805_HandSoldering, F.Cu at (153.1, 156.5)
- added R75: 470, Resistors_SMD:R_0805_HandSoldering, F.Cu at (157.8, 150.9)
- added R76: 470, Resistors_SMD:R_0805_HandSoldering, F.Cu at (153.1, 158.4)
- added R77: 470, Resistors_SMD:R_0805_HandSoldering, F.Cu at (157.8, 152.8)
- added R78: 470, Resistors_SMD:R_0805_HandSoldering, F.Cu at (153.1, 154.6)
- added R79: 470, Resistors_SMD:R_0805_HandSoldering, F.Cu at (162.6, 151.0)
- added R8: 2k, Resistors_SMD:R_0805_HandSoldering, F.Cu at (200.7, 135.3)
- added R80: 470, Resistors_SMD:R_0805_HandSoldering, F.Cu at (226.6, 108.4)
- added R81: 470, Resistors_SMD:R_0805_HandSoldering, F.Cu at (218.9, 127.5)
- added R82: 2k, Resistors_SMD:R_0805_HandSoldering, F.Cu at (191.1, 153.9)
- added R83: 2k, Resistors_SMD:R_0805_HandSoldering, F.Cu at (210.2, 133.1)
- added R84: 2k, Resistors_SMD:R_0805_HandSoldering, F.Cu at (210.2, 135.0)
- added R85: 2k, Resistors_SMD:R_0805_HandSoldering, F.Cu at (195.8, 150.3)
- added R86: 2k, Resistors_SMD:R_0805_HandSoldering, F.Cu at (223.7, 123.7)
- added R87: 2k, Resistors_SMD:R_0805_HandSoldering, F.Cu at (226.6, 119.7)
- added R88: 2k, Resistors_SMD:R_0805_HandSoldering, F.Cu at (205.5, 140.5)
- added R89: 2k, Resistors_SMD:R_0805_HandSoldering, F.Cu at (205.5, 142.4)
- added R9: 2k, Resistors_SMD:R_0805_HandSoldering, F.Cu at (226.6, 110.3)
- added R90: 470, Resistors_SMD:R_0805_HandSoldering, F.Cu at (210.2, 136.8)
- added R91: 470, Resistors_SMD:R_0805_HandSoldering, F.Cu at (191.1, 155.8)
- added R92: 470, Resistors_SMD:R_0805_HandSoldering, F.Cu at (231.3, 115.9)
- added R93: 470, Resistors_SMD:R_0805_HandSoldering, F.Cu at (200.7, 146.6)
- added R94: 470, Resistors_SMD:R_0805_HandSoldering, F.Cu at (210.2, 140.6)
- added U1: Acc, Housings_QFP:TQFP-44_10x10mm_Pitch0.8mm, F.Cu at (204.0, 114.2)
- added U10: PC_H, Housings_QFP:TQFP-44_10x10mm_Pitch0.8mm, F.Cu at (182.1, 141.1)
- added U11: RAM_Page, Housings_QFP:TQFP-44_10x10mm_Pitch0.8mm, F.Cu at (217.5, 114.2)
- added U2: X, Housings_QFP:TQFP-44_10x10mm_Pitch0.8mm, F.Cu at (182.1, 127.6)
- added U3: IR, Housings_QFP:TQFP-44_10x10mm_Pitch0.8mm, F.Cu at (168.7, 141.4)
- added U4: Multiplexer, Housings_QFP:TQFP-44_10x10mm_Pitch0.8mm, F.Cu at (190.6, 114.2)
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
Commit message: Reduce num pages to 64
Parts:
- J11: value Conn_01x05 -> Page
- J9: value Conn_01x05 -> Index
Connections:
- U11 pad 12: (no net) -> /D6
- U11 pad 13: (no net) -> /D7
- U11 pad 14: (no net) -> /AIDX0
- U11 pad 16: (no net) -> /AIDX2
- U11 pad 18: (no net) -> /AIDX1
- U11 pad 19: (no net) -> /AIDX3
- U11 pad 2: (no net) -> /D0
- U11 pad 20: (no net) -> /AIDX4
- U11 pad 21: (no net) -> /AIDX5
- U11 pad 22: (no net) -> /AIDX6
- U11 pad 23: (no net) -> /AIDX7
- U11 pad 27: (no net) -> /AIDX8
- U11 pad 28: (no net) -> /AIDX9
- U11 pad 29: (no net) -> /AIDX10
- U11 pad 3: (no net) -> /D1
- U11 pad 30: (no net) -> /AIDX11
- U11 pad 43: (no net) -> /RAM_WE
- U11 pad 44: (no net) -> /RAM_OE
- U11 pad 5: (no net) -> /D2
- U11 pad 6: (no net) -> /D3
- U11 pad 7: (no net) -> /D4
- U11 pad 8: (no net) -> /D5
- U4 pad 18: (no net) -> /X0
- U4 pad 19: (no net) -> /X1
- U4 pad 20: (no net) -> /X2
- U4 pad 21: (no net) -> /X3
- U4 pad 22: (no net) -> /X4
- U4 pad 23: (no net) -> /X5
- U4 pad 27: (no net) -> /X6
- U4 pad 28: (no net) -> /X7
- U5 pad 2: (no net) -> /RAM_OE
- U5 pad 23: (no net) -> /IDX_EN
- U5 pad 3: (no net) -> /RAM_WE
- U9 pad 1: (no net) -> /IDX_EN
- U9 pad 12: (no net) -> /ADDR6
- U9 pad 13: (no net) -> /ADDR7
- U9 pad 14: (no net) -> /ADDR8
- U9 pad 16: (no net) -> /ADDR9
- U9 pad 18: (no net) -> /ADDR10
- U9 pad 19: (no net) -> /ADDR11
- U9 pad 2: (no net) -> /ADDR0
- U9 pad 20: (no net) -> /X0
- U9 pad 21: (no net) -> /X1
- U9 pad 22: (no net) -> /X2
- U9 pad 23: (no net) -> /X3
- U9 pad 27: (no net) -> /X4
- U9 pad 28: (no net) -> /X5
- U9 pad 29: (no net) -> /X6
- U9 pad 3: (no net) -> /ADDR1
- U9 pad 30: (no net) -> /X7
- U9 pad 31: (no net) -> /AIDX0
- U9 pad 32: (no net) -> /AIDX1
- U9 pad 34: (no net) -> /AIDX2
- U9 pad 36: (no net) -> /AIDX3
- U9 pad 37: (no net) -> /AIDX4
- U9 pad 38: (no net) -> /AIDX5
- U9 pad 39: (no net) -> /AIDX6
- U9 pad 40: (no net) -> /AIDX7
- U9 pad 41: (no net) -> /AIDX8
- U9 pad 42: (no net) -> /AIDX9
- U9 pad 43: (no net) -> /AIDX10
- U9 pad 44: (no net) -> /AIDX11
- U9 pad 5: (no net) -> /ADDR2
- U9 pad 6: (no net) -> /ADDR3
- U9 pad 7: (no net) -> /ADDR4
- U9 pad 8: (no net) -> /ADDR5

Commit message: Add RAM
Parts:
- added C34: 100n, Capacitors_SMD:C_0805_HandSoldering, F.Cu at (268.7, 130.6)
- added C35: 100n, Capacitors_SMD:C_0805_HandSoldering, F.Cu at (251.1, 145.6)
- added C36: 100n, Capacitors_SMD:C_0805_HandSoldering, F.Cu at (273.1, 126.8)
- added C37: 100n, Capacitors_SMD:C_0805_HandSoldering, F.Cu at (263.8, 136.2)
- added C38: 100n, Capacitors_SMD:C_0805_HandSoldering, F.Cu at (280.5, 117.4)
- added C39: 100n, Capacitors_SMD:C_0805_HandSoldering, F.Cu at (277.5, 123.0)
- added C40: 100n, Capacitors_SMD:C_0805_HandSoldering, F.Cu at (257.4, 141.8)
- added C41: 100n, Capacitors_SMD:C_0805_HandSoldering, F.Cu at (263.2, 132.5)
- added D100: LED_Small, LEDs:LED_0805_HandSoldering, F.Cu at (219.9, 130.4)
- added D101: LED_Small, LEDs:LED_0805_HandSoldering, F.Cu at (248.4, 111.8)
- added D102: LED_Small, LEDs:LED_0805_HandSoldering, F.Cu at (227.8, 124.8)
- added D103: LED_Small, LEDs:LED_0805_HandSoldering, F.Cu at (236.9, 115.5)
- added D104: LED_Small, LEDs:LED_0805_HandSoldering, F.Cu at (205.6, 113.7)
- added D105: LED_Small, LEDs:LED_0805_HandSoldering, F.Cu at (213.3, 177.3)
- added D106: LED_Small, LEDs:LED_0805_HandSoldering, F.Cu at (222.9, 174.8)
- added D107: LED_Small, LEDs:LED_0805_HandSoldering, F.Cu at (208.9, 126.7)
- added D108: LED_Small, LEDs:LED_0805_HandSoldering, F.Cu at (191.1, 119.2)
- added D109: LED_Small, LEDs:LED_0805_HandSoldering, F.Cu at (234.9, 72.4)
- added D110: LED_Small, LEDs:LED_0805_HandSoldering, F.Cu at (191.4, 121.1)
- added D111: LED_Small, LEDs:LED_0805_HandSoldering, F.Cu at (186.4, 124.8)
- added D112: LED_Small, LEDs:LED_0805_HandSoldering, F.Cu at (203.7, 115.5)
- added D113: LED_Small, LEDs:LED_0805_HandSoldering, F.Cu at (189.4, 126.6)
- added D114: LED_Small, LEDs:LED_0805_HandSoldering, F.Cu at (210.3, 111.8)
- added D115: LED_Small, LEDs:LED_0805_HandSoldering, F.Cu at (244.9, 78.0)
- added D116: LED_Small, LEDs:LED_0805_HandSoldering, F.Cu at (213.9, 134.1)
- added D117: LED_Small, LEDs:LED_0805_HandSoldering, F.Cu at (198.2, 145.2)
- added D118: LED_Small, LEDs:LED_0805_HandSoldering, F.Cu at (202.9, 171.2)
- added D119: LED_Small, LEDs:LED_0805_HandSoldering, F.Cu at (208.4, 141.5)
- added D120: LED_Small, LEDs:LED_0805_HandSoldering, F.Cu at (195.2, 182.4)
- added D121: LED_Small, LEDs:LED_0805_HandSoldering, F.Cu at (248.9, 113.7)
- added D122: LED_Small, LEDs:LED_0805_HandSoldering, F.Cu at (218.8, 132.3)
- added D123: LED_Small, LEDs:LED_0805_HandSoldering, F.Cu at (237.4, 117.4)
- added D124: LED_Small, LEDs:LED_0805_HandSoldering, F.Cu at (255.8, 110.0)
- added D53: LED_Small, LEDs:LED_0805_HandSoldering, F.Cu at (255.9, 89.2)
- added D54: LED_Small, LEDs:LED_0805_HandSoldering, F.Cu at (219.6, 121.2)
- added D55: LED_Small, LEDs:LED_0805_HandSoldering, F.Cu at (231.1, 111.8)
- added D56: LED_Small, LEDs:LED_0805_HandSoldering, F.Cu at (207.3, 130.4)
- added D57: LED_Small, LEDs:LED_0805_HandSoldering, F.Cu at (228.9, 115.5)
- added D58: LED_Small, LEDs:LED_0805_HandSoldering, F.Cu at (215.5, 123.0)
- added D59: LED_Small, LEDs:LED_0805_HandSoldering, F.Cu at (225.6, 117.4)
- added D60: LED_Small, LEDs:LED_0805_HandSoldering, F.Cu at (194.6, 174.8)
- added D61: LED_Small, LEDs:LED_0805_HandSoldering, F.Cu at (202.9, 134.1)
- added D62: LED_Small, LEDs:LED_0805_HandSoldering, F.Cu at (203.4, 136.0)
- added D63: LED_Small, LEDs:LED_0805_HandSoldering, F.Cu at (185.6, 143.4)
- added D64: LED_Small, LEDs:LED_0805_HandSoldering, F.Cu at (190.5, 145.2)
- added D65: LED_Small, LEDs:LED_0805_HandSoldering, F.Cu at (195.5, 139.7)
- added D66: LED_Small, LEDs:LED_0805_HandSoldering, F.Cu at (199.6, 137.8)
- added D67: LED_Small, LEDs:LED_0805_HandSoldering, F.Cu at (196.0, 141.5)
- added D68: LED_Small, LEDs:LED_0805_HandSoldering, F.Cu at (214.4, 130.4)
- added D69: LED_Small, LEDs:LED_0805_HandSoldering, F.Cu at (224.3, 126.6)
- added D70: LED_Small, LEDs:LED_0805_HandSoldering, F.Cu at (201.8, 143.4)
- added D71: LED_Small, LEDs:LED_0805_HandSoldering, F.Cu at (215.8, 126.7)
- added D72: LED_Small, LEDs:LED_0805_HandSoldering, F.Cu at (208.1, 132.3)
- added D73: LED_Small, LEDs:LED_0805_HandSoldering, F.Cu at (230.6, 113.7)
- added D74: LED_Small, LEDs:LED_0805_HandSoldering, F.Cu at (223.4, 123.0)
- added D75: LED_Small, LEDs:LED_0805_HandSoldering, F.Cu at (212.5, 128.6)
- added D76: LED_Small, LEDs:LED_0805_HandSoldering, F.Cu at (241.5, 110.0)
- added D77: LED_Small, LEDs:LED_0805_HandSoldering, F.Cu at (226.2, 119.2)
- added D78: LED_Small, LEDs:LED_0805_HandSoldering, F.Cu at (264.2, 80.5)
- added D79: LED_Small, LEDs:LED_0805_HandSoldering, F.Cu at (224.0, 121.1)
- added D80: LED_Small, LEDs:LED_0805_HandSoldering, F.Cu at (238.5, 111.8)
- added D81: LED_Small, LEDs:LED_0805_HandSoldering, F.Cu at (208.4, 178.1)
- added D82: LED_Small, LEDs:LED_0805_HandSoldering, F.Cu at (228.1, 113.7)
- added D83: LED_Small, LEDs:LED_0805_HandSoldering, F.Cu at (217.4, 124.9)
- added D84: LED_Small, LEDs:LED_0805_HandSoldering, F.Cu at (234.4, 115.5)
- added D85: LED_Small, LEDs:LED_0805_HandSoldering, F.Cu at (204.8, 134.1)
- added D86: LED_Small, LEDs:LED_0805_HandSoldering, F.Cu at (183.3, 173.5)
- added D87: LED_Small, LEDs:LED_0805_HandSoldering, F.Cu at (191.9, 143.4)
- added D88: LED_Small, LEDs:LED_0805_HandSoldering, F.Cu at (199.9, 139.7)
- added D89: LED_Small, LEDs:LED_0805_HandSoldering, F.Cu at (195.2, 145.2)
- added D90: LED_Small, LEDs:LED_0805_HandSoldering, F.Cu at (207.0, 136.0)
- added D91: LED_Small, LEDs:LED_0805_HandSoldering, F.Cu at (231.9, 117.4)
- added D92: LED_Small, LEDs:LED_0805_HandSoldering, F.Cu at (215.2, 124.9)
- added D93: LED_Small, LEDs:LED_0805_HandSoldering, F.Cu at (216.0, 137.8)
- added D94: LED_Small, LEDs:LED_0805_HandSoldering, F.Cu at (223.7, 122.9)
- added D95: LED_Small, LEDs:LED_0805_HandSoldering, F.Cu at (245.7, 110.0)
- added D96: LED_Small, LEDs:LED_0805_HandSoldering, F.Cu at (220.4, 128.6)
- added D97: LED_Small, LEDs:LED_0805_HandSoldering, F.Cu at (218.0, 126.7)
- added D98: LED_Small, LEDs:LED_0805_HandSoldering, F.Cu at (251.3, 53.3)
- added D99: LED_Small, LEDs:LED_0805_HandSoldering, F.Cu at (231.4, 121.1)
- added J12: Conn_02x16_Odd_Even, Pin_Headers:Pin_Header_Straight_2x16_Pitch2.54mm, F.Cu at (-6.10, 196.3)
- added J13: Page, Pin_Headers:Pin_Header_Straight_1x05_Pitch2.54mm, F.Cu at (81.0, 180.3)
- added J14: Conn_02x16_Odd_Even, Pin_Headers:Pin_Header_Straight_2x16_Pitch2.54mm, F.Cu at (6.10, 196.3)
- added R100: 2k, Resistors_SMD:R_0805_HandSoldering, F.Cu at (228.4, 147.3)
- added R101: 2k, Resistors_SMD:R_0805_HandSoldering, F.Cu at (275.3, 110.0)
- added R102: 2k, Resistors_SMD:R_0805_HandSoldering, F.Cu at (253.6, 128.7)
- added R103: 2k, Resistors_SMD:R_0805_HandSoldering, F.Cu at (233.3, 132.3)
- added R104: 2k, Resistors_SMD:R_0805_HandSoldering, F.Cu at (270.9, 121.3)
- added R105: 2k, Resistors_SMD:R_0805_HandSoldering, F.Cu at (258.0, 130.7)
- added R106: 2k, Resistors_SMD:R_0805_HandSoldering, F.Cu at (279.1, 111.9)
- added R107: 470, Resistors_SMD:R_0805_HandSoldering, F.Cu at (264.8, 125.0)
- added R108: 470, Resistors_SMD:R_0805_HandSoldering, F.Cu at (237.7, 143.7)
- added R109: 470, Resistors_SMD:R_0805_HandSoldering, F.Cu at (252.2, 134.4)
- added R110: 470, Resistors_SMD:R_0805_HandSoldering, F.Cu at (274.7, 115.6)
- added R111: 470, Resistors_SMD:R_0805_HandSoldering, F.Cu at (266.2, 126.9)
- added R112: 470, Resistors_SMD:R_0805_HandSoldering, F.Cu at (252.0, 136.3)
- added R113: 470, Resistors_SMD:R_0805_HandSoldering, F.Cu at (237.2, 145.6)
- added R114: 470, Resistors_SMD:R_0805_HandSoldering, F.Cu at (264.6, 130.7)
- added R115: 2k, Resistors_SMD:R_0805_HandSoldering, F.Cu at (278.0, 113.8)
- added R116: 2k, Resistors_SMD:R_0805_HandSoldering, F.Cu at (236.3, 149.2)
- added R117: 2k, Resistors_SMD:R_0805_HandSoldering, F.Cu at (272.0, 123.2)
- added R118: 2k, Resistors_SMD:R_0805_HandSoldering, F.Cu at (248.7, 141.8)
- added R119: 2k, Resistors_SMD:R_0805_HandSoldering, F.Cu at (233.6, 151.1)
- added R120: 2k, Resistors_SMD:R_0805_HandSoldering, F.Cu at (281.0, 110.0)
- added R121: 2k, Resistors_SMD:R_0805_HandSoldering, F.Cu at (275.8, 119.4)
- added R122: 2k, Resistors_SMD:R_0805_HandSoldering, F.Cu at (242.1, 147.5)
- added R123: 470, Resistors_SMD:R_0805_HandSoldering, F.Cu at (251.7, 138.1)
- added R124: 470, Resistors_SMD:R_0805_HandSoldering, F.Cu at (265.4, 128.8)
- added R125: 470, Resistors_SMD:R_0805_HandSoldering, F.Cu at (275.0, 117.5)
- added R126: 470, Resistors_SMD:R_0805_HandSoldering, F.Cu at (200.1, 124.8)
- added R127: 470, Resistors_SMD:R_0805_HandSoldering, F.Cu at (222.1, 110.0)
- added R128: 470, Resistors_SMD:R_0805_HandSoldering, F.Cu at (211.4, 113.7)
- added R129: 470, Resistors_SMD:R_0805_HandSoldering, F.Cu at (187.3, 132.2)
- added R130: 470, Resistors_SMD:R_0805_HandSoldering, F.Cu at (190.8, 128.5)
- added R131: 470, Resistors_SMD:R_0805_HandSoldering, F.Cu at (205.4, 117.4)
- added R132: 470, Resistors_SMD:R_0805_HandSoldering, F.Cu at (200.7, 122.9)
- added R133: 470, Resistors_SMD:R_0805_HandSoldering, F.Cu at (204.0, 119.3)
- added R134: 470, Resistors_SMD:R_0805_HandSoldering, F.Cu at (101.5, 173.2)
- added R135: 470, Resistors_SMD:R_0805_HandSoldering, F.Cu at (204.5, 121.1)
- added R136: 470, Resistors_SMD:R_0805_HandSoldering, F.Cu at (225.4, 145.4)
- added R137: 470, Resistors_SMD:R_0805_HandSoldering, F.Cu at (214.1, 115.6)
- added R138: 470, Resistors_SMD:R_0805_HandSoldering, F.Cu at (200.4, 126.7)
- added R139: 470, Resistors_SMD:R_0805_HandSoldering, F.Cu at (191.6, 130.4)
- added R140: 470, Resistors_SMD:R_0805_HandSoldering, F.Cu at (190.0, 134.1)
- added R141: 470, Resistors_SMD:R_0805_HandSoldering, F.Cu at (222.9, 111.9)
- added R142: 2k, Resistors_SMD:R_0805_HandSoldering, F.Cu at (189.2, 135.9)
- added R143: 2k, Resistors_SMD:R_0805_HandSoldering, F.Cu at (187.8, 137.8)
- added R144: 2k, Resistors_SMD:R_0805_HandSoldering, F.Cu at (222.6, 113.7)
- added R145: 2k, Resistors_SMD:R_0805_HandSoldering, F.Cu at (197.1, 132.2)
- added R146: 2k, Resistors_SMD:R_0805_HandSoldering, F.Cu at (247.0, 140.0)
- added R147: 2k, Resistors_SMD:R_0805_HandSoldering, F.Cu at (227.6, 149.2)
- added R148: 2k, Resistors_SMD:R_0805_HandSoldering, F.Cu at (238.8, 141.8)
- added R149: 2k, Resistors_SMD:R_0805_HandSoldering, F.Cu at (265.7, 123.2)
- added R150: 2k, Resistors_SMD:R_0805_HandSoldering, F.Cu at (278.6, 110.0)
- added R151: 2k, Resistors_SMD:R_0805_HandSoldering, F.Cu at (261.8, 128.8)
- added R152: 2k, Resistors_SMD:R_0805_HandSoldering, F.Cu at (271.7, 119.4)
- added R153: 2k, Resistors_SMD:R_0805_HandSoldering, F.Cu at (244.8, 138.1)
- added R154: 2k, Resistors_SMD:R_0805_HandSoldering, F.Cu at (233.0, 147.4)
- added R155: 2k, Resistors_SMD:R_0805_HandSoldering, F.Cu at (261.3, 132.6)
- added R156: 2k, Resistors_SMD:R_0805_HandSoldering, F.Cu at (270.6, 125.0)
- added R157: 2k, Resistors_SMD:R_0805_HandSoldering, F.Cu at (281.6, 111.9)
- added R158: 2k, Resistors_SMD:R_0805_HandSoldering, F.Cu at (234.7, 130.4)
- added R159: 2k, Resistors_SMD:R_0805_HandSoldering, F.Cu at (241.8, 151.2)
- added R160: 1.2k, Resistors_SMD:R_0805_HandSoldering, F.Cu at (274.4, 123.2)
- added R161: 1.2k, Resistors_SMD:R_0805_HandSoldering, F.Cu at (281.3, 113.8)
- added R162: 1.2k, Resistors_SMD:R_0805_HandSoldering, F.Cu at (278.3, 117.5)
- added R163: 1.2k, Resistors_SMD:R_0805_HandSoldering, F.Cu at (277.7, 115.6)
- added R164: 1.2k, Resistors_SMD:R_0805_HandSoldering, F.Cu at (259.4, 136.3)
- added R165: 1.2k, Resistors_SMD:R_0805_HandSoldering, F.Cu at (258.5, 134.4)
- added R166: 1.2k, Resistors_SMD:R_0805_HandSoldering, F.Cu at (270.3, 126.9)
- added R167: 1.2k, Resistors_SMD:R_0805_HandSoldering, F.Cu at (246.8, 145.6)
- added R168: 1.2k, Resistors_SMD:R_0805_HandSoldering, F.Cu at (246.2, 143.7)
- added R169: 1.2k, Resistors_SMD:R_0805_HandSoldering, F.Cu at (280.8, 108.1)
- added R170: 1.2k, Resistors_SMD:R_0805_HandSoldering, F.Cu at (252.5, 141.9)
- added R171: 1.2k, Resistors_SMD:R_0805_HandSoldering, F.Cu at (256.1, 140.0)
- added R172: 1.2k, Resistors_SMD:R_0805_HandSoldering, F.Cu at (240.4, 149.3)
- added R173: 2k, Resistors_SMD:R_0805_HandSoldering, F.Cu at (274.2, 121.3)
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Connections:
- C29 pad 1: VCC -> GND
- C29 pad 2: GND -> VCC
- R1 pad 1: /IR0 -> /D0
- R1 pad 2: Net-(D1-Pad2) -> Net-(D25-Pad2)
- R10 pad 1: /A1 -> /RAM_WE
- R10 pad 2: Net-(D10-Pad2) -> Net-(D2-Pad2)
- R11 pad 1: /A2 -> /PC_OE
- R11 pad 2: Net-(D11-Pad2) -> Net-(D3-Pad2)
- R12 pad 1: /A3 -> /ALU_OE
- R12 pad 2: Net-(D12-Pad2) -> Net-(D4-Pad2)
- R13 pad 1: /A4 -> /ALU_WE
- R13 pad 2: Net-(D13-Pad2) -> Net-(D5-Pad2)
- R14 pad 1: /A5 -> /A_OE
- R14 pad 2: Net-(D14-Pad2) -> Net-(D6-Pad2)
- R15 pad 1: /A6 -> /A_WE
- R15 pad 2: Net-(D15-Pad2) -> Net-(D7-Pad2)
- R16 pad 1: /A7 -> /X_OE
- R16 pad 2: Net-(D16-Pad2) -> Net-(D8-Pad2)
- R17 pad 1: /AC -> /X_WE
- R17 pad 2: Net-(D17-Pad2) -> Net-(D9-Pad2)
- R18 pad 1: /X0 -> /IR_OE
- R18 pad 2: Net-(D18-Pad2) -> Net-(D10-Pad2)
- R19 pad 1: /X1 -> /IR_WE
- R19 pad 2: Net-(D19-Pad2) -> Net-(D11-Pad2)
- R2 pad 1: /IR1 -> /D1
- R2 pad 2: Net-(D2-Pad2) -> Net-(D26-Pad2)
- R20 pad 1: /X2 -> /AR_OE
- R20 pad 2: Net-(D20-Pad2) -> Net-(D12-Pad2)
- R21 pad 1: /X3 -> /AR_WE
- R21 pad 2: Net-(D21-Pad2) -> Net-(D13-Pad2)
- R22 pad 1: /X4 -> /PC_INC
- R22 pad 2: Net-(D22-Pad2) -> Net-(D14-Pad2)
- R23 pad 1: /X5 -> /IDX_EN
- R23 pad 2: Net-(D23-Pad2) -> Net-(D15-Pad2)
- R24 pad 1: /X6 -> /A_Z
- R24 pad 2: Net-(D24-Pad2) -> Net-(D16-Pad2)
- R25 pad 1: /X7 -> /IR0
- R25 pad 2: Net-(D25-Pad2) -> Net-(D17-Pad2)
- R26 pad 1: /D1 -> /IR1
- R26 pad 2: Net-(R26-Pad2) -> Net-(D18-Pad2)
- R27 pad 1: /D0 -> /IR2
- R27 pad 2: Net-(R27-Pad2) -> Net-(D19-Pad2)
- R28 pad 1: /D2 -> /IR3
- R28 pad 2: Net-(R28-Pad2) -> Net-(D20-Pad2)
- R29 pad 1: /D3 -> /IR4
- R29 pad 2: Net-(R29-Pad2) -> Net-(D21-Pad2)
- R3 pad 1: /IR2 -> /D2
- R3 pad 2: Net-(D3-Pad2) -> Net-(D27-Pad2)
- R30 pad 1: /D4 -> /IR5
- R30 pad 2: Net-(R30-Pad2) -> Net-(D22-Pad2)
- R31 pad 1: /D5 -> /IR6
- R31 pad 2: Net-(R31-Pad2) -> Net-(D23-Pad2)
- R32 pad 1: /D6 -> /IR7
- R32 pad 2: Net-(R32-Pad2) -> Net-(D24-Pad2)
- R33 pad 1: /D7 -> /A0
- R33 pad 2: Net-(R33-Pad2) -> Net-(D33-Pad2)
- R34 pad 1: /D1 -> /A1
- R34 pad 2: Net-(R34-Pad2) -> Net-(D34-Pad2)
- R35 pad 1: /D0 -> /A2
- R35 pad 2: Net-(R35-Pad2) -> Net-(D35-Pad2)
- R36 pad 1: /D2 -> /A3
- R36 pad 2: Net-(R36-Pad2) -> Net-(D36-Pad2)
- R37 pad 1: /D3 -> /A4
- R37 pad 2: Net-(R37-Pad2) -> Net-(D37-Pad2)
- R38 pad 1: /D4 -> /A5
- R38 pad 2: Net-(R38-Pad2) -> Net-(D38-Pad2)
- R39 pad 1: /D5 -> /A6
- R39 pad 2: Net-(R39-Pad2) -> Net-(D39-Pad2)
- R4 pad 1: /IR3 -> /D3
- R4 pad 2: Net-(D4-Pad2) -> Net-(D28-Pad2)
- R40 pad 1: /D6 -> /A7
- R40 pad 2: Net-(R40-Pad2) -> Net-(D40-Pad2)
- R41 pad 1: /D7 -> /AC
- R41 pad 2: Net-(R41-Pad2) -> Net-(D41-Pad2)
- R42 pad 1: /ADDR9 -> /X0
- R42 pad 2: Net-(R42-Pad2) -> Net-(D42-Pad2)
- R43 pad 1: /ADDR8 -> /X1
- R43 pad 2: Net-(R43-Pad2) -> Net-(D43-Pad2)
- R44 pad 1: /ADDR10 -> /X2
- R44 pad 2: Net-(R44-Pad2) -> Net-(D44-Pad2)
- R45 pad 1: /ADDR11 -> /X3
- R45 pad 2: Net-(R45-Pad2) -> Net-(D45-Pad2)
- R46 pad 1: /ADDR12 -> /X4
- R46 pad 2: Net-(R46-Pad2) -> Net-(D46-Pad2)
- R47 pad 1: /AR0 -> /X5
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
Commit message: Fix base_addr
Parts:
- moved C6 111.2 mm to (142.5, 122.9)
Changed lines of the file:
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@@
   )
   (module Capacitors_SMD:C_0805_HandSoldering (layer F.Cu)
-    (at 250.043401 151.038001)
+    (at 142.474 122.936)
     (descr "Capacitor SMD 0805, hand soldering")
     (tags "capacitor 0805")

Commit message: Lay PCB, most parts except busses
Parts:
- moved J12 430.1 mm to (416.6, 116.8)
- moved J14 292.5 mm to (281.9, 99.1)
- moved C8 260.3 mm to (35.6, 213.4), turned to 270 degrees
- moved R58 256.8 mm to (17.8, 127.0)
- moved R56 254.8 mm to (17.8, 72.4)
- moved R54 252.6 mm to (17.8, 67.3)
- moved R59 249.3 mm to (17.8, 129.5)
- moved R50 249.2 mm to (17.8, 57.1)
- moved R24 245.8 mm to (20.3, 35.6), turned to 90 degrees
- moved C3 245.5 mm to (40.6, 45.7), turned to 90 degrees
- moved R63 245.0 mm to (17.8, 139.7)
- moved C1 243.8 mm to (35.6, 71.1), turned to 270 degrees
- moved R55 243.7 mm to (17.8, 69.8)
- moved R41 243.4 mm to (25.4, 35.6), turned to 90 degrees
- moved R70 242.5 mm to (20.3, 180.3)
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Routing:
- net VCC: track 0.00 -> 219.6 mm
- net /A_Z: track 0.00 -> 27.2 mm
- net /X0: track 0.00 -> 23.1 mm
- net Net-(R115-Pad1): track 0.00 -> 23.1 mm
- net /IR0: track 0.00 -> 23.1 mm
- net /A0: track 0.00 -> 23.1 mm
- net /AR0: track 0.00 -> 23.1 mm
- net Net-(R99-Pad1): track 0.00 -> 23.1 mm
- net /ALU0: track 0.00 -> 23.1 mm
- net /A1: track 0.00 -> 22.9 mm
- net /X1: track 0.00 -> 22.9 mm
- net /ALU1: track 0.00 -> 22.9 mm
- net /IR1: track 0.00 -> 22.9 mm
- net Net-(R100-Pad1): track 0.00 -> 22.9 mm
- net /AR1: track 0.00 -> 22.9 mm
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Other:
- net class Default: clearance 0.2 -> 0.254; trace_width 0.25 -> 0.254
- rule trace_clearance: 0.2 -> 0.254
- board text added: "0"
- board text added: "1"
- board text added: "10"
- board text added: "11"
- board text added: "12"
- board text added: "2"
- board text added: "3"
- board text added: "4"
- board text added: "5"
- board text added: "6"
- board text added: "7"
- board text added: "8"
- board text added: "9"
- board text added: "ALU"
- board text added: "Accumulator (A)"
- board text added: "Address (AR)"
- board text added: "C"
- board text added: "Decoder"
- board text added: "EN"
- board text added: "GPIO & RNG"
- board text added: "INC OE"
- board text added: "Index (X)"
- board text added: "Instruction (IR)"
- board text added: "Memory Index"
- board text added: "Memory Page"
- board text added: "Program Counter (PC)"
- board text added: "RAM (256kiB)"
- board text added: "WE OE"
- board text added: "Z"

Commit message: routing a/x/alu
Parts:
- moved C11 10.2 mm to (96.5, 61.0)
- moved C21 10.2 mm to (121.9, 45.7)
- moved D63 10.2 mm to (124.5, 30.5)
- moved D64 10.2 mm to (121.9, 30.5)
- moved J4 10.2 mm to (69.8, 53.3)
- moved R92 10.2 mm to (124.5, 35.6)
- moved R93 10.2 mm to (121.9, 35.6)
- moved U4 10.2 mm to (83.8, 58.4)
- moved C10 10.2 mm to (81.3, 71.1)
- moved C12 10.2 mm to (86.4, 45.7)
- moved C19 10.2 mm to (116.8, 71.1)
- moved C20 10.2 mm to (132.1, 61.0)
- moved D4 10.2 mm to (132.1, 73.7)
- moved D5 10.2 mm to (132.1, 71.1)
- moved D61 10.2 mm to (129.5, 30.5)
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Routing:
- net /X7: track 18.6 -> 114.2 mm, vias 0 -> 2
- net /AC: track 22.9 -> 116.7 mm, vias 0 -> 2
- net /X6: track 17.9 -> 108.3 mm, vias 0 -> 2
- net /X5: track 17.2 -> 101.1 mm, vias 0 -> 2
- net /X4: track 17.9 -> 96.6 mm, vias 0 -> 2
- net /X3: track 22.6 -> 98.2 mm, vias 0 -> 2
- net /X2: track 22.8 -> 95.9 mm, vias 0 -> 2
- net /X1: track 22.9 -> 92.3 mm, vias 0 -> 2
- net /X0: track 23.1 -> 89.4 mm, vias 0 -> 2
- net /A7: track 18.6 -> 78.8 mm, vias 0 -> 2
- net /A6: track 17.9 -> 75.9 mm, vias 0 -> 2
- net /A5: track 17.2 -> 73.0 mm, vias 0 -> 2
- net /A4: track 17.9 -> 71.8 mm, vias 0 -> 2
- net /ALUA4: track 0.00 -> 42.8 mm
- net /ALUA7: track 0.00 -> 41.0 mm, vias 0 -> 2
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Other:
- net class Default: via_dia 0.8 -> 0.75

Commit message: VHDL for ioregister and program_counter.
Parts:
- moved C14 12.7 mm to (96.5, 124.5)
- moved R80 12.7 mm to (83.8, 99.1)
- moved D59 12.7 mm to (83.8, 94.0)
- moved J5 12.7 mm to (69.8, 116.8)
- moved U5 12.7 mm to (83.8, 121.9)
- moved C13 12.7 mm to (81.3, 134.6)
- moved C15 12.7 mm to (86.4, 109.2)
- moved R79 12.7 mm to (86.4, 99.1)
- moved R81 12.7 mm to (81.3, 99.1)
- moved D58 12.7 mm to (86.4, 94.0)
- moved D60 12.7 mm to (81.3, 94.0)
- moved R57 1.27 mm to (17.8, 73.7)
- moved R50 1.27 mm to (17.8, 55.9)
- moved R51 1.27 mm to (17.8, 58.4)
- moved R52 1.27 mm to (17.8, 61.0)
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Connections:
- U1 pad 28: (no net) -> Net-(U1-Pad28)
- U1 pad 34: (no net) -> Net-(U1-Pad34)
- U1 pad 36: (no net) -> Net-(U1-Pad36)
- U10 pad 40: (no net) -> Net-(U10-Pad40)
- U10 pad 41: (no net) -> Net-(U10-Pad41)
- U10 pad 42: (no net) -> Net-(U10-Pad42)
- U11 pad 12: (no net) -> Net-(U11-Pad12)
- U11 pad 13: (no net) -> Net-(U11-Pad13)
- U11 pad 14: (no net) -> Net-(U11-Pad14)
- U11 pad 22: (no net) -> Net-(U11-Pad22)
- U11 pad 23: (no net) -> Net-(U11-Pad23)
- U11 pad 27: (no net) -> Net-(U11-Pad27)
- U11 pad 28: (no net) -> Net-(U11-Pad28)
- U11 pad 34: (no net) -> Net-(U11-Pad34)
- U11 pad 36: (no net) -> Net-(U11-Pad36)
- U11 pad 41: (no net) -> Net-(U11-Pad41)
- U11 pad 42: (no net) -> Net-(U11-Pad42)
- U11 pad 8: (no net) -> Net-(U11-Pad8)
- U2 pad 1: (no net) -> Net-(U2-Pad1)
- U2 pad 14: (no net) -> Net-(U2-Pad14)
- U2 pad 28: (no net) -> Net-(U2-Pad28)
- U2 pad 34: (no net) -> Net-(U2-Pad34)
- U2 pad 36: (no net) -> Net-(U2-Pad36)
- U2 pad 41: (no net) -> Net-(U2-Pad41)
- U2 pad 42: (no net) -> Net-(U2-Pad42)
- U3 pad 1: (no net) -> Net-(U3-Pad1)
- U3 pad 14: (no net) -> Net-(U3-Pad14)
- U3 pad 22: (no net) -> Net-(U3-Pad22)
- U3 pad 23: (no net) -> Net-(U3-Pad23)
- U3 pad 27: (no net) -> Net-(U3-Pad27)
- U3 pad 28: (no net) -> Net-(U3-Pad28)
- U3 pad 34: (no net) -> Net-(U3-Pad34)
- U3 pad 36: (no net) -> Net-(U3-Pad36)
- U3 pad 41: (no net) -> Net-(U3-Pad41)
- U3 pad 42: (no net) -> Net-(U3-Pad42)
- U4 pad 1: (no net) -> Net-(U4-Pad1)
- U4 pad 2: (no net) -> Net-(U4-Pad2)
- U4 pad 3: (no net) -> Net-(U4-Pad3)
- U4 pad 34: (no net) -> Net-(U4-Pad34)
- U4 pad 36: (no net) -> Net-(U4-Pad36)
- U4 pad 41: (no net) -> Net-(U4-Pad41)
- U4 pad 42: (no net) -> Net-(U4-Pad42)
- U4 pad 44: (no net) -> Net-(U4-Pad44)
- U5 pad 1: (no net) -> Net-(U5-Pad1)
- U5 pad 28: (no net) -> /AC
- U5 pad 34: (no net) -> Net-(U5-Pad34)
- U5 pad 36: (no net) -> Net-(U5-Pad36)
- U5 pad 37: (no net) -> Net-(U5-Pad37)
- U5 pad 38: (no net) -> Net-(U5-Pad38)
- U5 pad 42: (no net) -> Net-(U5-Pad42)
- U5 pad 43: (no net) -> Net-(U5-Pad43)
- U5 pad 44: (no net) -> Net-(U5-Pad44)
- U6 pad 1: (no net) -> Net-(U6-Pad1)
- U6 pad 14: (no net) -> Net-(U6-Pad14)
- U6 pad 28: (no net) -> Net-(U6-Pad28)
- U6 pad 34: (no net) -> Net-(U6-Pad34)
- U6 pad 36: (no net) -> Net-(U6-Pad36)
- U6 pad 41: (no net) -> Net-(U6-Pad41)
- U6 pad 42: (no net) -> Net-(U6-Pad42)
- U7 pad 1: (no net) -> Net-(U7-Pad1)
- U7 pad 34: (no net) -> Net-(U7-Pad34)
- U7 pad 36: (no net) -> Net-(U7-Pad36)
- U7 pad 42: (no net) -> Net-(U7-Pad42)
- U9 pad 14: (no net) -> Net-(U9-Pad14)
- U9 pad 28: (no net) -> Net-(U9-Pad28)
- U9 pad 34: (no net) -> Net-(U9-Pad34)
- U9 pad 36: (no net) -> Net-(U9-Pad36)
- U9 pad 41: (no net) -> Net-(U9-Pad41)
Routing:
- net /ALU3: track 22.6 -> 209.4 mm, vias 0 -> 4
- net /ALU2: track 22.8 -> 208.2 mm, vias 0 -> 4
- net /ALU7: track 18.6 -> 203.9 mm, vias 0 -> 4
- net /ALU6: track 17.9 -> 202.8 mm, vias 0 -> 4
- net /ALU1: track 22.9 -> 205.1 mm, vias 0 -> 4
- net /ALU5: track 17.2 -> 199.3 mm, vias 0 -> 4
- net /ALU0: track 23.1 -> 203.6 mm, vias 0 -> 4
- net /ALU4: track 17.9 -> 198.1 mm, vias 0 -> 4
- net /ALU8: track 22.9 -> 116.8 mm, vias 0 -> 4
- net Net-(R65-Pad2): track 0.00 -> 41.8 mm, vias 0 -> 2
- net Net-(R57-Pad2): track 0.00 -> 40.7 mm, vias 0 -> 2
- net /A_CC: track 0.00 -> 38.5 mm, vias 0 -> 1
- net /A_Z: track 27.2 -> 64.3 mm, vias 0 -> 1
- net Net-(R56-Pad2): track 0.00 -> 36.2 mm, vias 0 -> 2
- net Net-(R64-Pad2): track 0.00 -> 35.7 mm, vias 0 -> 2
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Other:
- board outline added: 264.2 x 190.5 mm
- copper layers 2 -> 4
