File: hardware/cpld-cpu.sch (KiCad schematic (older format))
At the start: 44 parts

Commit message: Most of the schematic done (just missing RAM/mmappedio)
Parts:
- removed U?: Decoder, Housings_QFP:TQFP-44_10x10mm_Pitch0.8mm, symbol CPLD_CPU_Component:CPLD_CPU_Decoder
- added D1, D10, D11, D12, D13, D14, D15, D16, D17, D18, D19, D2, D20, D21, D22, D23, D24, D25, D26, D27, D28, D29, D3, D30, D31, D32, D33, D34, D35, D36, D37, D38, D39, D4, D40, D41, D42, D43, D44, D45, D46, D47, D48, D49, D5, D50, D51, D52, D6, D7, D8, D9: LED_Small, LEDs:LED_0805_HandSoldering, symbol Device:LED_Small
- added J1: Acc, Pin_Headers:Pin_Header_Straight_1x05_Pitch2.54mm, symbol Connector_Generic:Conn_01x05
- added J10: PC_H, Pin_Headers:Pin_Header_Straight_1x05_Pitch2.54mm, symbol Connector_Generic:Conn_01x05
- added J11, J9: Conn_01x05, Pin_Headers:Pin_Header_Straight_1x05_Pitch2.54mm, symbol Connector_Generic:Conn_01x05
- added J2: X, Pin_Headers:Pin_Header_Straight_1x05_Pitch2.54mm, symbol Connector_Generic:Conn_01x05
- added J3: IR, Pin_Headers:Pin_Header_Straight_1x05_Pitch2.54mm, symbol Connector_Generic:Conn_01x05
- added J4: AXM, Pin_Headers:Pin_Header_Straight_1x05_Pitch2.54mm, symbol Connector_Generic:Conn_01x05
- added J5: Dec, Pin_Headers:Pin_Header_Straight_1x05_Pitch2.54mm, symbol Connector_Generic:Conn_01x05
- added J6: AR, Pin_Headers:Pin_Header_Straight_1x05_Pitch2.54mm, symbol Connector_Generic:Conn_01x05
- added J7: ALU, Pin_Headers:Pin_Header_Straight_1x05_Pitch2.54mm, symbol Connector_Generic:Conn_01x05
- added J8: PC_L, Pin_Headers:Pin_Header_Straight_1x05_Pitch2.54mm, symbol Connector_Generic:Conn_01x05
- added R1, R10, R11, R12, R13, R14, R15, R16, R17, R18, R19, R2, R20, R21, R22, R23, R24, R25, R3, R4, R47, R48, R49, R5, R50, R51, R52, R53, R54, R55, R56, R57, R6, R66, R67, R68, R69, R7, R70, R71, R72, R73, R8, R82, R83, R84, R85, R86, R87, R88, R89, R9: 2k, Resistors_SMD:R_0805_HandSoldering, symbol Device:R_Small
- added R26, R27, R28, R29, R30, R31, R32, R33, R34, R35, R36, R37, R38, R39, R40, R41, R42, R43, R44, R45, R46, R58, R59, R60, R61, R62, R63, R64, R65, R74, R75, R76, R77, R78, R79, R80, R81, R90, R91, R92, R93, R94: 470, Resistors_SMD:R_0805_HandSoldering, symbol Device:R_Small
- added U5: Decoder, Housings_QFP:TQFP-44_10x10mm_Pitch0.8mm, symbol CPLD_CPU_Component:CPLD_CPU_Decoder
- C1, C10, C11, C12, C13, C14, C15, C16, C17, C18, C19, C2, C20, C21, C22, C23, C24, C25, C26, C27, C28, C29, C3, C30, C31, C32, C33, C4, C5, C6, C7, C8, C9: renamed from C?; footprint (none) -> Capacitors_SMD:C_0805_HandSoldering
- gave numbers to parts that had none: 10
Connections:
- net GND: now also D1.1 (K), D10.1 (K), D11.1 (K), D12.1 (K), D13.1 (K), D14.1 (K), D15.1 (K), D16.1 (K), D17.1 (K), D18.1 (K), D19.1 (K), D2.1 (K), D20.1 (K), D21.1 (K), D22.1 (K), D23.1 (K), D24.1 (K), D25.1 (K), D26.1 (K), D27.1 (K), D28.1 (K), D29.1 (K), D3.1 (K), D30.1 (K), D31.1 (K), D32.1 (K), D33.1 (K), D34.1 (K), D35.1 (K), D36.1 (K), D37.1 (K), D38.1 (K), D39.1 (K), D4.1 (K), D40.1 (K), D41.1 (K), D42.1 (K), D43.1 (K), D44.1 (K), D45.1 (K), D46.1 (K), D47.1 (K), D48.1 (K), D49.1 (K), D5.1 (K), D50.1 (K), D51.1 (K), D52.1 (K), D6.1 (K), D7.1 (K), D8.1 (K), D9.1 (K), J1.5 (Pin_5), J10.5 (Pin_5), J11.5 (Pin_5), J2.5 (Pin_5), J3.5 (Pin_5), J4.5 (Pin_5), J5.5 (Pin_5), J6.5 (Pin_5), J7.5 (Pin_5), J8.5 (Pin_5), J9.5 (Pin_5), U5.17 (GND), U5.25 (GND), U5.4 (GND)
- net VCC: now also U5.15 (VCC), U5.26 (VCCIO), U5.35 (VCC)
- net A_CC: now reaches U1.1 (P1/GCK3/CC)
- net A_CC: now also U5.29 (P29/CC)
- net at U1.10 (TMS): now also J1.2 (Pin_2)
- net at U1.11 (TCK): now also J1.3 (Pin_3)
- net ALU6: now reaches U1.12 (P12/IN6)
- net ALU6: now also U2.12 (P12/IN6), U7.39 (P39/OUT6)
- net ALU7: now reaches U1.13 (P13/IN7)
- net ALU7: now also U2.13 (P13/IN7), U7.40 (P40/OUT7)
- net ALU8: now reaches U1.14 (P14/IN8)
- net ALU8: now also U7.41 (P41/OUT8)
- net at U1.16 (P16/OUT0): now also R27.2
- net at U1.18 (P18/OUT1): now also R26.2
- net at U1.19 (P19/OUT2): now also R28.2
- net ALU0: now reaches U1.2 (P2/IN0)
- net ALU0: now also U2.2 (P2/IN0), U7.29 (P29/OUT0)
- net at U1.20 (P20/OUT3): now also R29.2
- net at U1.21 (P21/OUT4): now also R30.2
- net at U1.22 (P22/OUT5): now also R31.2
- net at U1.23 (P23/OUT6): now also R32.2
- net at U1.24 (TDO): now also J1.4 (Pin_4)
- net at U1.27 (P27/OUT7): now also R33.2
- net A0: now reaches U1.29 (P29/ST0)
- net A0: now also U4.5 (P5/A0), R9.1
- net ALU1: now reaches U1.3 (P3/IN1)
- net ALU1: now also U2.3 (P3/IN1), U7.30 (P30/OUT1)
- net A1: now reaches U1.30 (P30/ST1)
- net A1: now also U4.6 (P6/A1), R10.1
- net A2: now reaches U1.31 (P31/ST2)
- net A2: now also U4.7 (P7/A2), R11.1
- net A3: now reaches U1.32 (P32/ST3)
- net A3: now also U4.8 (P8/A3), R12.1
- net RST: now reaches U1.33 (P33/GSR/~RST)
- net RST: now also U10.33 (P33/GSR/~RST), U11.33 (P33/GSR/~RST), U2.33 (P33/GSR/~RST), U3.33 (P33/GSR/~RST), U4.33 (P33/GSR/~RST), U6.33 (P33/GSR/~RST), U7.33 (P33/GSR/~RST), U8.33 (P33/GSR/~RST), U9.33 (P33/GSR/~RST), U5.33 (P33/GSR/~RST)
- net A4: now reaches U1.37 (P37/ST4)
- net A4: now also U4.12 (P12/A4), R13.1
- net A5: now reaches U1.38 (P38/ST5)
- net A5: now also U4.13 (P13/A5), R14.1
- net A6: now reaches U1.39 (P39/ST6)
- net A6: now also U4.14 (P14/A6), R15.1
- net A7: now reaches U1.40 (P40/ST7)
- net A7: now also U4.16 (P16/A7), R16.1
- net AC: now reaches U1.41 (P41/ST8)
- net AC: now also U7.14 (P14/A8), R17.1
- net A_Z: now reaches U1.42 (P42/Z)
- net A_Z: now also U5.27 (P27/Z)
- net A_WE: now reaches U1.43 (P43/GCK1/WE)
- net A_WE: now also U5.13 (P13/A_WE)
- net A_OE: now reaches U1.44 (P44/GCK2/OE)
- net A_OE: now also U5.12 (P12/A_OE)
- net ALU2: now reaches U1.5 (P5/IN2)
- net ALU2: now also U2.5 (P5/IN2), U7.31 (P31/OUT2)
- net ALU3: now reaches U1.6 (P6/IN3)
- net ALU3: now also U2.6 (P6/IN3), U7.32 (P32/FN)
- net ALU4: now reaches U1.7 (P7/IN4)
- net ALU4: now also U2.7 (P7/IN4), U7.37 (P37/B0)
- net ALU5: now reaches U1.8 (P8/IN5)
- net ALU5: now also U2.8 (P8/IN5), U7.38 (P38/B1)
- net at U1.9 (TDI): now also J1.1 (Pin_1)
- net at U7.10 (TMS): now also J7.2 (Pin_2)
- net at U7.11 (TCK): now also J7.3 (Pin_3)
- net ALUA6: now reaches U7.12 (P12/A6)
- net ALUA6: now also U4.39 (P39/OUT6)
- net ALUA7: now reaches U7.13 (P13/A7)
- net ALUA7: now also U4.40 (P40/OUT7)
- net D0: now reaches U7.16 (P16/OUT3)
- net D0: now also U3.2 (P2/IN0), U6.2 (P2/IN0), R27.1, R35.1
- net D1: now reaches U7.18 (P18/OUT4)
- net D1: now also U3.3 (P3/IN1), U6.3 (P3/IN1), R26.1, R34.1
- net D2: now reaches U7.19 (P19/B2)
- net D2: now also U3.5 (P5/IN2), U6.5 (P5/IN2), R28.1, R36.1
- net ALUA0: now reaches U7.2 (P2/A0)
- net ALUA0: now also U4.29 (P29/OUT0)
- net D3: now reaches U7.20 (P20/B3)
- net D3: now also U3.6 (P6/IN3), U6.6 (P6/IN3), R29.1, R37.1
- net D4: now reaches U7.21 (P21/B4)
- net D4: now also U3.7 (P7/IN4), U6.7 (P7/IN4), R30.1, R38.1
- net D5: now reaches U7.22 (P22/B5)
- net D5: now also U3.8 (P8/IN5), U6.8 (P8/IN5), R31.1, R39.1
- net D6: now reaches U7.23 (P23/B6)
- net D6: now also U3.12 (P12/IN6), U6.12 (P12/IN6), R32.1, R40.1
- net at U7.24 (TDO): now also J7.4 (Pin_4)
- net D7: now reaches U7.27 (P27/B7)
- net D7: now also U3.13 (P13/IN7), U6.13 (P13/IN7), R33.1, R41.1
- net IR5: now reaches U7.28 (P28/OUT5)
- net IR5: now also U3.38 (P38/ST5), R6.1, U5.39 (P39/INSTR0)
- net ALUA1: now reaches U7.3 (P3/A1)
- net ALUA1: now also U4.30 (P30/OUT1)
- net ALU_OE: now reaches U7.43 (P43/GCK1/WE)
- net ALU_OE: now also U5.7 (P7/ALU_OE)
- net ALU_WE: now reaches U7.44 (P44/GCK2/OE)
- net ALU_WE: now also U5.8 (P8/ALU_WE)
- net ALUA2: now reaches U7.5 (P5/A2)
- net ALUA2: now also U4.31 (P31/OUT2)
- net ALUA3: now reaches U7.6 (P6/A3)
- net ALUA3: now also U4.32 (P32/OUT3)
- net ALUA4: now reaches U7.7 (P7/A4)
- net ALUA4: now also U4.37 (P37/OUT4)
- net ALUA5: now reaches U7.8 (P8/A5)
- net ALUA5: now also U4.38 (P38/OUT5)
- net at U7.9 (TDI): now also J7.1 (Pin_1)
- net at U4.10 (TMS): now also J4.2 (Pin_2)
- net at U4.11 (TCK): now also J4.3 (Pin_3)
- net X0: now reaches U4.18 (P18/B0)
- net X0: now also U2.29 (P29/ST0), U9.20 (P20/X0), R18.1
- net X1: now reaches U4.19 (P19/B1)
- net X1: now also U2.30 (P30/ST1), U9.21 (P21/X1), R19.1
- net X2: now reaches U4.20 (P20/B2)
- net X2: now also U2.31 (P31/ST2), U9.22 (P22/X2), R20.1
- net X3: now reaches U4.21 (P21/B3)
- net X3: now also U2.32 (P32/ST3), U9.23 (P23/X3), R21.1
- net X4: now reaches U4.22 (P22/B4)
- net X4: now also U2.37 (P37/ST4), U9.27 (P27/X4), R22.1
- net X5: now reaches U4.23 (P23/B5)
- net X5: now also U2.38 (P38/ST5), U9.28 (P28/X5), R23.1
- net at U4.24 (TDO): now also J4.4 (Pin_4)
- net X6: now reaches U4.27 (P27/B6)
- net X6: now also U2.39 (P39/ST6), U9.29 (P29/X6), R24.1
- net X7: now reaches U4.28 (P28/B7)
- net X7: now also U2.40 (P40/ST7), U9.30 (P30/X7), R25.1
- net IR7: now reaches U4.43 (P43/GCK1/SEL)
- net IR7: now also U3.40 (P40/ST7), R8.1, U5.41 (P41/INSTR2)
- net at U4.9 (TDI): now also J4.1 (Pin_1)
- net IDX_EN: now reaches U9.1 (P1/GCK3/EN)
- net IDX_EN: now also U5.23 (P23/IDX_EN)
- net at U9.10 (TMS): now also J9.2 (Pin_2)
- net at U9.11 (TCK): now also J9.3 (Pin_3)
- net ADDR6: now reaches U9.12 (P12/A6)
- net ADDR6: now also R64.1, R80.1
- net ADDR7: now reaches U9.13 (P13/A7)
- net ADDR7: now also R65.1, R81.1
- net ADDR8: now reaches U9.14 (P14/A8)
- net ADDR8: now also R43.1, R91.1
- net ADDR9: now reaches U9.16 (P16/A9)
- net ADDR9: now also R42.1, R90.1
- net ADDR10: now reaches U9.18 (P18/10)
- net ADDR10: now also R44.1, R92.1
- net ADDR11: now reaches U9.19 (P19/A11)
- net ADDR11: now also R45.1, R93.1
- net at U9.24 (TDO): now also J9.4 (Pin_4)
- net ADDR2: now reaches U9.5 (P5/A2)
- net ADDR2: now also R60.1, R76.1
- net ADDR3: now reaches U9.6 (P6/A3)
- net ADDR3: now also R61.1, R77.1
- net ADDR4: now reaches U9.7 (P7/A4)
- net ADDR4: now also R62.1, R78.1
- net ADDR5: now reaches U9.8 (P8/A5)
- net ADDR5: now also R63.1, R79.1
- net at U9.9 (TDI): now also J9.1 (Pin_1)
- net at U11.10 (TMS): now also J11.2 (Pin_2)
- net at U11.11 (TCK): now also J11.3 (Pin_3)
- net at U11.24 (TDO): now also J11.4 (Pin_4)
- net at U11.9 (TDI): now also J11.1 (Pin_1)
- net at U2.10 (TMS): now also J2.2 (Pin_2)
- net at U2.11 (TCK): now also J2.3 (Pin_3)
- net at U2.16 (P16/OUT0): now also R35.2
- net at U2.18 (P18/OUT1): now also R34.2
- net at U2.19 (P19/OUT2): now also R36.2
- net at U2.20 (P20/OUT3): now also R37.2
- net at U2.21 (P21/OUT4): now also R38.2
- net at U2.22 (P22/OUT5): now also R39.2
- net at U2.23 (P23/OUT6): now also R40.2
- net at U2.24 (TDO): now also J2.4 (Pin_4)
- net at U2.27 (P27/OUT7): now also R41.2
- net X_WE: now reaches U2.43 (P43/GCK1/WE)
- net X_WE: now also U5.18 (P18/X_WE)
- net X_OE: now reaches U2.44 (P44/GCK2/OE)
- net X_OE: now also U5.14 (P14/X_OE)
- net at U2.9 (TDI): now also J2.1 (Pin_1)
- net at U3.10 (TMS): now also J3.2 (Pin_2)
- net at U3.11 (TCK): now also J3.3 (Pin_3)
- net at U3.16 (P16/OUT0): now also R43.2
- net at U3.18 (P18/OUT1): now also R42.2
- net at U3.19 (P19/OUT2): now also R44.2
- net at U3.20 (P20/OUT3): now also R45.2
- net at U3.21 (P21/OUT4): now also R46.2
- net at U3.24 (TDO): now also J3.4 (Pin_4)
- net IR0: now reaches U3.29 (P29/ST0)
- net IR0: now also U10.2 (P2/IN0), R1.1
- net IR1: now reaches U3.30 (P30/ST1)
- net IR1: now also U10.3 (P3/IN1), R2.1
- net IR2: now reaches U3.31 (P31/ST2)
- net IR2: now also U10.5 (P5/IN2), R3.1
- net IR3: now reaches U3.32 (P32/ST3)
- net IR3: now also U10.6 (P6/IN3), R4.1
- net IR4: now reaches U3.37 (P37/ST4)
- net IR4: now also U10.7 (P7/IN4), R5.1
- net IR6: now reaches U3.39 (P39/ST6)
- net IR6: now also R7.1, U5.40 (P40/INSTR1)
- net IR_WE: now reaches U3.43 (P43/GCK1/WE)
- net IR_WE: now also U5.19 (P19/IR_WE)
- net IR_OE: now reaches U3.44 (P44/GCK2/OE)
- net IR_OE: now also U5.16 (P16/IR_OE)
- net at U3.9 (TDI): now also J3.1 (Pin_1)
- net at U6.10 (TMS): now also J6.2 (Pin_2)
- net at U6.11 (TCK): now also J6.3 (Pin_3)
- net at U6.16 (P16/OUT0): now also R59.2
- net at U6.18 (P18/OUT1): now also R58.2
- net at U6.19 (P19/OUT2): now also R60.2
- net at U6.20 (P20/OUT3): now also R61.2
- net at U6.21 (P21/OUT4): now also R62.2
- net at U6.22 (P22/OUT5): now also R63.2
- net at U6.23 (P23/OUT6): now also R64.2
- net at U6.24 (TDO): now also J6.4 (Pin_4)
- net at U6.27 (P27/OUT7): now also R65.2
- net AR0: now reaches U6.29 (P29/ST0)
- net AR0: now also U8.2 (P2/IN0), R47.1
- net AR1: now reaches U6.30 (P30/ST1)
- net AR1: now also U8.3 (P3/IN1), R48.1
- net AR2: now reaches U6.31 (P31/ST2)
- net AR2: now also U8.5 (P5/IN2), R49.1
- net AR3: now reaches U6.32 (P32/ST3)
- net AR3: now also U8.6 (P6/IN3), R50.1
- net AR4: now reaches U6.37 (P37/ST4)
- net AR4: now also U8.7 (P7/IN4), R51.1
- net AR5: now reaches U6.38 (P38/ST5)
- net AR5: now also U8.8 (P8/IN5), R52.1
- net AR6: now reaches U6.39 (P39/ST6)
- net AR6: now also U8.12 (P12/IN6), R53.1
- net AR7: now reaches U6.40 (P40/ST7)
- net AR7: now also U8.13 (P13/IN7), R54.1
- net AR_WE: now reaches U6.43 (P43/GCK1/WE)
- net AR_WE: now also U5.21 (P21/AR_WE)
- net AR_OE: now reaches U6.44 (P44/GCK2/OE)
- net AR_OE: now also U5.20 (P20/AR_OE)
- net at U6.9 (TDI): now also J6.1 (Pin_1)
- net PC_INC: now reaches U8.1 (P1/GCK3/INC)
- net PC_INC: now also U5.22 (P22/PC_INC)
- net at U8.10 (TMS): now also J8.2 (Pin_2)
- net at U8.11 (TCK): now also J8.3 (Pin_3)
- net at U8.16 (P16/OUT0): now also R75.2
- net at U8.18 (P18/OUT1): now also R74.2
- net at U8.19 (P19/OUT2): now also R76.2
- net at U8.20 (P20/OUT3): now also R77.2
- net at U8.21 (P21/OUT4): now also R78.2
- net at U8.22 (P22/OUT5): now also R79.2
- net at U8.23 (P23/OUT6): now also R80.2
- net at U8.24 (TDO): now also J8.4 (Pin_4)
- net at U8.27 (P27/OUT7): now also R81.2
- net at U8.29 (P29/ST0): now also R66.1
- net at U8.30 (P30/ST1): now also R67.1
- net at U8.31 (P31/ST2): now also R68.1
- net at U8.32 (P32/ST3): now also R69.1
- net at U8.37 (P37/ST4): now also R70.1
- net at U8.38 (P38/ST5): now also R71.1
- net at U8.39 (P39/ST6): now also R72.1
- net at U8.40 (P40/ST7): now also R73.1
- net PC_CARRY: now reaches U10.1 (P1/GCK3/INC), U8.42 (P42/CARRY)
- net PC_WE: now reaches U8.43 (P43/GCK1/WE)
- net PC_WE: now also U10.43 (P43/GCK1/WE), U5.6 (P6/PC_WE)
- net PC_OE: now reaches U8.44 (P44/GCK2/OE)
- net PC_OE: now also U10.44 (P44/GCK2/OE), U5.5 (P5/PC_OE)
- net at U8.9 (TDI): now also J8.1 (Pin_1)
- net at U10.10 (TMS): now also J10.2 (Pin_2)
- net at U10.11 (TCK): now also J10.3 (Pin_3)
- net at U10.16 (P16/OUT0): now also R91.2
- net at U10.18 (P18/OUT1): now also R90.2
- net at U10.19 (P19/OUT2): now also R92.2
- net at U10.20 (P20/OUT3): now also R93.2
- net at U10.21 (P21/OUT4): now also R94.2
- net at U10.24 (TDO): now also J10.4 (Pin_4)
- net at U10.29 (P29/ST0): now also R82.1
- net at U10.30 (P30/ST1): now also R83.1
- net at U10.31 (P31/ST2): now also R84.1
- net at U10.32 (P32/ST3): now also R85.1
- net at U10.37 (P37/ST4): now also R86.1
- net at U10.38 (P38/ST5): now also R87.1
- net at U10.39 (P39/ST6): now also R88.1
- net at U10.40 (P40/ST7): now also R89.1
- net at U10.9 (TDI): now also J10.1 (Pin_1)
- new net: D37.2 (A), R66.2
- new net: D38.2 (A), R67.2
- new net: D39.2 (A), R68.2
- new net: D40.2 (A), R69.2
- new net: D41.2 (A), R70.2
- new net: D42.2 (A), R71.2
- new net: D43.2 (A), R72.2
- new net: D44.2 (A), R73.2
- new net: D45.2 (A), R82.2
- new net: D46.2 (A), R83.2
- new net: D47.2 (A), R84.2
- new net: D48.2 (A), R85.2
- new net: D49.2 (A), R86.2
- new net: D50.2 (A), R87.2
- new net: D51.2 (A), R88.2
- new net: D52.2 (A), R89.2
- new net: J5.1 (Pin_1), U5.9 (TDI)
- new net: J5.2 (Pin_2), U5.10 (TMS)
- new net: J5.3 (Pin_3), U5.11 (TCK)
- new net: J5.4 (Pin_4), U5.24 (TDO)
- new net: D26.2 (A), R47.2
- new net: D27.2 (A), R48.2
- new net: D28.2 (A), R49.2
- new net: D29.2 (A), R50.2
- new net: D30.2 (A), R51.2
- new net: D31.2 (A), R52.2
- new net: D32.2 (A), R53.2
- new net: D33.2 (A), R54.2
- new net: D1.2 (A), R1.2
- new net: D2.2 (A), R2.2
- new net: D3.2 (A), R3.2
- new net: D4.2 (A), R4.2
- new net: D5.2 (A), R5.2
- new net: D6.2 (A), R6.2
- new net: D7.2 (A), R7.2
- new net: D8.2 (A), R8.2
- new net: R55.1, U5.30 (P30/ST0)
- new net: R56.1, U5.31 (P31/ST1)
- new net: R57.1, U5.32 (P32/ST2)
- new net: D34.2 (A), R55.2
- new net: D35.2 (A), R56.2
- new net: D36.2 (A), R57.2
- new net: D9.2 (A), R9.2
- new net: D10.2 (A), R10.2
- new net: D11.2 (A), R11.2
- new net: D12.2 (A), R12.2
- new net: D13.2 (A), R13.2
- new net: D14.2 (A), R14.2
- new net: D15.2 (A), R15.2
- new net: D16.2 (A), R16.2
- new net: D17.2 (A), R17.2
- new net: D18.2 (A), R18.2
- new net: D19.2 (A), R19.2
- new net: D20.2 (A), R20.2
- new net: D21.2 (A), R21.2
- new net: D22.2 (A), R22.2
- new net: D23.2 (A), R23.2
- new net: D24.2 (A), R24.2
- new net: D25.2 (A), R25.2
- new net ADDR0: R59.1, R75.1
- new net ADDR1: R58.1, R74.1
- new net ADDR12: R46.1, R94.1
- new net RAM_OE: U5.2 (P2/RAM_OE)
- new net RAM_WE: U5.3 (P3/RAM_WE)
- no-connect marks 0 -> 64
Other:
- moved on the sheet: C1, C10, C11, C12, C13, C14, C15, C16, C17, C18, C19, C2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

Commit message: Ram connections
Parts:
- J11: value Conn_01x05 -> Page
- J9: value Conn_01x05 -> Index
Connections:
- net ADDR0: now also U9.2 (P2/A0)
- net ADDR1: now also U9.3 (P3/A1)
- net D0: now also U11.2 (P2/PROG1)
- net D1: now also U11.3 (P3/PROG2)
- net D2: now also U11.5 (P5/D4)
- net D3: now also U11.6 (P6/D5)
- net D4: now also U11.7 (P7/D6)
- net D5: now also U11.8 (P8/D7)
- net D6: now also U11.12 (P12/A0)
- net D7: now also U11.13 (P13/A1)
- net RAM_OE: now also U11.44 (P44/GCK2)
- net RAM_WE: now also U11.43 (P43/GCK1/WE)
- net AIDX0: now reaches U9.31 (P31/OUT0)
- net AIDX0: now also U11.14 (P14/A2)
- net AIDX1: now reaches U9.32 (P32/OUT1)
- net AIDX1: now also U11.18 (P18/A4)
- net AIDX2: now reaches U9.34 (P34/GTS2/OUT2)
- net AIDX2: now also U11.16 (P16/A3)
- net AIDX3: now reaches U9.36 (P36/GTS1/OUT3)
- net AIDX3: now also U11.19 (P19/A5)
- net AIDX4: now reaches U9.37 (P37/OUT4)
- net AIDX4: now also U11.20 (P20/A6)
- net AIDX5: now reaches U9.38 (P38/OUT5)
- net AIDX5: now also U11.21 (P21/A7)
- net AIDX6: now reaches U9.39 (P39/OUT6)
- net AIDX6: now also U11.22 (P22/A8)
- net AIDX7: now reaches U9.40 (P40/OUT7)
- net AIDX7: now also U11.23 (P23/A9)
- net AIDX8: now reaches U9.41 (P41/OUT8)
- net AIDX8: now also U11.27 (P27/A10)
- net AIDX9: now reaches U9.42 (P42/OUT9)
- net AIDX9: now also U11.28 (P28/A11)
- net AIDX10: now reaches U9.43 (P43/GCK1/OUT10)
- net AIDX10: now also U11.29 (P29/A12)
- net AIDX11: now reaches U9.44 (P44/GCK2/OUT11)
- net AIDX11: now also U11.30 (P30/Z)
- no-connect marks 64 -> 65
Other:
- moved on the sheet: C31, C32, C33, J11, U11

Commit message: Reduce num pages to 64
Parts:
- added D? (x46): LED_Small, LEDs:LED_0805_HandSoldering, symbol Device:LED_Small
- added R? (x6): 470, Resistors_SMD:R_0805_HandSoldering, symbol Device:R_Small
- added R? (x25): 2k, Resistors_SMD:R_0805_HandSoldering, symbol Device:R_Small
- added R? (x21): 1.2k, Resistors_SMD:R_0805_HandSoldering, symbol Device:R_Small
Connections:
- net ADDR0: now also R?.1
- net ADDR1: now also R?.1
- net ADDR10: now also R?.1
- net ADDR11: now also R?.1
- net ADDR12: now also U11.1 (P1/GCK3/PROG0), R?.1
- net ADDR2: now also R?.1
- net ADDR3: now also R?.1
- net ADDR4: now also R?.1
- net ADDR5: now also R?.1
- net ADDR6: now also R?.1
- net ADDR7: now also R?.1
- net ADDR8: now also R?.1
- net ADDR9: now also R?.1
- net AIDX0: now also U11.12 (P12/A0); no longer U11.14 (P14/A2)
- net AIDX1: now also U11.13 (P13/A1); no longer U11.18 (P18/A4)
- net AIDX10: now also U11.27 (P27/A10); no longer U11.29 (P29/A12)
- net AIDX11: now also U11.28 (P28/A11); no longer U11.30 (P30/Z)
- net AIDX2: now also U11.14 (P14/A2); no longer U11.16 (P16/A3)
- net AIDX3: now also U11.16 (P16/A3); no longer U11.19 (P19/A5)
- net AIDX4: now also U11.18 (P18/A4); no longer U11.20 (P20/A6)
- net AIDX5: now also U11.19 (P19/A5); no longer U11.21 (P21/A7)
- net AIDX6: now also U11.20 (P20/A6); no longer U11.22 (P22/A8)
- net AIDX7: now also U11.21 (P21/A7); no longer U11.23 (P23/A9)
- net AIDX8: now also U11.22 (P22/A8); no longer U11.27 (P27/A10)
- net AIDX9: now also U11.23 (P23/A9); no longer U11.28 (P28/A11)
- net ALU0: now also R?.1
- net ALU1: now also R?.1
- net ALU2: now also R?.1
- net ALU3: now also R?.1
- net ALU4: now also R?.1
- net ALU5: now also R?.1
- net ALU6: now also R?.1
- net ALU7: now also R?.1
- net ALU8: now also R?.1
- net ALU_OE: now also R?.1
- net ALU_WE: now also R?.1
- net AR_OE: now also R?.1
- net AR_WE: now also R?.1
- net A_OE: now also R?.1
- net A_WE: now also R?.1
- net A_Z: now also R?.1
- net D0: now also R?.1, R?.2; no longer U11.2 (P2/PROG1)
- net D1: now also R?.1, R?.2; no longer U11.3 (P3/PROG2)
- net D2: now also R?.1, R?.1; no longer U11.5 (P5/D4)
- net D3: now also R?.1, R?.1; no longer U11.6 (P6/D5)
- net D4: now also R?.1, R?.1; no longer U11.7 (P7/D6)
- net D5: now also R?.1, R?.1; no longer U11.8 (P8/D7)
- net D6: now also R?.1; no longer U11.12 (P12/A0)
- net D7: now also R?.1; no longer U11.13 (P13/A1)
- net GND: now also D?.1 (K), D?.1 (K), D?.1 (K), D?.1 (K), D?.1 (K), D?.1 (K), D?.1 (K), D?.1 (K), D?.1 (K), D?.1 (K), D?.1 (K), D?.1 (K), D?.1 (K), D?.1 (K), D?.1 (K), D?.1 (K), D?.1 (K), D?.1 (K), D?.1 (K), D?.1 (K), D?.1 (K), D?.1 (K), D?.1 (K), D?.1 (K), D?.1 (K), D?.1 (K), D?.1 (K), D?.1 (K), D?.1 (K), D?.1 (K), D?.1 (K), D?.1 (K), D?.1 (K), D?.1 (K), D?.1 (K), D?.1 (K), D?.1 (K), D?.1 (K), D?.1 (K), D?.1 (K), D?.1 (K), D?.1 (K), D?.1 (K), D?.1 (K), D?.1 (K), D?.1 (K)
- net IDX_EN: now also R?.1
- net IR_OE: now also R?.1
- net IR_WE: now also R?.1
- net PC_INC: now also R?.1
- net PC_OE: now also R?.1
- net RAM_OE: now also R?.1
- net RAM_WE: now also R?.1
- net X_OE: now also R?.1
- net X_WE: now also R?.1
- new net: R?.1, U11.2 (P2/PROG1)
- new net: R?.1, U11.3 (P3/PROG2)
- new net: R?.2, U11.5 (P5/D4)
- new net: R?.2, U11.6 (P6/D5)
- new net: R?.2, U11.7 (P7/D6)
- new net: R?.2, U11.8 (P8/D7)
- new net: D?.2 (A), R?.2 (x46)
- no-connect marks 65 -> 67
Other:
- moved on the sheet: D1, D2, D3, D4, D5, D6, D7, D8, R1, R2, R3, R4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

Commit message: Add RAM
Parts:
- added C28, C29, C36, C37, C38, C39, C40, C41: 100n, Capacitors_SMD:C_0805_HandSoldering, symbol Device:C_Small
- added D100, D101, D102, D103, D117, D118, D119, D120, D121, D122, D123, D124, D86, D87, D88, D89, D90, D91, D92, D93, D94, D95, D96, D97, D98, D99: LED_Small, LEDs:LED_0805_HandSoldering, symbol Device:LED_Small
- added J12: Conn_02x16_Odd_Even, Pin_Headers:Pin_Header_Straight_2x16_Pitch2.54mm, symbol Connector_Generic:Conn_02x14_Odd_Even
- added J13: Page, Pin_Headers:Pin_Header_Straight_1x05_Pitch2.54mm, symbol Connector_Generic:Conn_01x05
- added J14: Conn_02x16_Odd_Even, Pin_Headers:Pin_Header_Straight_2x16_Pitch2.54mm, symbol Connector_Generic:Conn_02x16_Odd_Even
- added R125, R126, R127, R128, R129, R130, R131, R132, R181, R182, R183, R184, R185, R186, R187, R188: 470, Resistors_SMD:R_0805_HandSoldering, symbol Device:R_Small
- added R142, R143, R144, R145, R146, R147, R148, R149, R150, R151, R152, R153, R154, R155, R156, R157, R158, R159, R173, R174, R175, R176, R177, R178, R179, R180: 2k, Resistors_SMD:R_0805_HandSoldering, symbol Device:R_Small
- added R189, R190, R191: 10k, Resistors_SMD:R_0805_HandSoldering, symbol Device:R_Small
- added SW1, SW2, SW3: BTN0, Buttons_Switches_SMD:SW_SPST_B3S-1000, symbol Switch:SW_Push
- added U12: CY62138FV30LL, Housings_SSOP:TSOP-II-32_21.0x10.2mm_Pitch1.27mm, symbol CPLD_CPU_Component:CY62138FV30LL
- added U13: GPIO_RNG, Housings_QFP:TQFP-44_10x10mm_Pitch0.8mm, symbol CPLD_CPU_Component:CPLD_CPU_GPIO_RNG
- gave numbers to parts that had none: 98
- renumbered C25 to C22, C26 to C23, C27 to C24, C22 to C25, C23 to C26, C24 to C27, C31 to C30, C32 to C31, C33 to C32, C28 to C33, C29 to C34, C30 to C35, D1 to D17, D2 to D18, D3 to D19, D4 to D20, D5 to D21, D6 to D22, D7 to D23, D8 to D24, D9 to D33, D10 to D34, D11 to D35, D12 to D36, D13 to D37, D14 to D38, D15 to D39, D16 to D40, D17 to D41, D18 to D42, D19 to D43, D20 to D44, D21 to D45, D22 to D46, D23 to D47, D24 to D48, D25 to D49, D26 to D50, D27 to D51, D28 to D52, D29 to D53, D30 to D54, D31 to D55, D32 to D56, D33 to D57, D34 to D58, D35 to D59, D36 to D60, D37 to D70, D38 to D71, D39 to D72, D40 to D73, D41 to D74, D42 to D75, D43 to D76, D44 to D77, D45 to D78, D46 to D79, D47 to D80, D48 to D81, D49 to D82, D50 to D83, D51 to D84, D52 to D85, J11 to J10, J10 to J11, J9 to J8, J8 to J9, R67 to R100, R68 to R101, R69 to R102, R70 to R103, R71 to R104, R72 to R105, R73 to R106, R74 to R107, R75 to R108, R76 to R109, R77 to R110, R78 to R111, R79 to R112, R80 to R113, R81 to R114, R82 to R115, R83 to R116, R84 to R117, R85 to R118, R86 to R119, R87 to R120, R88 to R121, R89 to R122, R90 to R137, R91 to R138, R92 to R139, R93 to R140, R94 to R141, R1 to R25, R2 to R26, R3 to R27, R4 to R28, R5 to R29, R6 to R30, R7 to R31, R8 to R32, R9 to R33, R10 to R34, R11 to R35, R12 to R36, R13 to R37, R14 to R38, R15 to R39, R16 to R40, R17 to R41, R18 to R42, R19 to R43, R20 to R44, R21 to R45, R22 to R46, R23 to R47, R24 to R48, R25 to R49, R26 to R50, R27 to R51, R28 to R52, R29 to R53, R30 to R54, R31 to R55, R32 to R56, R33 to R57, R34 to R58, R35 to R59, R36 to R60, R37 to R61, R38 to R62, R39 to R63, R40 to R64, R41 to R65, R42 to R66, R43 to R67, R44 to R68, R45 to R69, R46 to R70, R47 to R71, R48 to R72, R49 to R73, R50 to R74, R51 to R75, R52 to R76, R53 to R77, R54 to R78, R55 to R79, R56 to R80, R57 to R81, R58 to R82, R59 to R83, R60 to R84, R61 to R85, R62 to R86, R63 to R87, R64 to R88, R65 to R89, R66 to R99, U11 to U10, U10 to U11, U9 to U8, U8 to U9
Connections:
- net D0: now also J14.1 (Pin_1), R125.2, R181.2
- net D1: now also J14.3 (Pin_3), R126.2, R182.2
- net D2: now also J14.5 (Pin_5), R127.2, R183.1
- net D3: now also J14.7 (Pin_7), R132.1, R184.1
- net D4: now also J14.9 (Pin_9), R131.1, R185.1
- net D5: now also J14.11 (Pin_11), R130.1, R186.1
- net D6: now also J14.13 (Pin_13), R129.1, R187.1
- net D7: now also J14.15 (Pin_15), R128.1, R188.1
- net GND: now also C28.2, C29.1, C36.2, C37.2, C38.2, C39.2, C40.2, C41.2, D100.1 (K), D101.1 (K), D102.1 (K), D103.1 (K), D117.1 (K), D118.1 (K), D119.1 (K), D120.1 (K), D121.1 (K), D122.1 (K), D123.1 (K), D124.1 (K), D86.1 (K), D87.1 (K), D88.1 (K), D89.1 (K), D90.1 (K), D91.1 (K), D92.1 (K), D93.1 (K), D94.1 (K), D95.1 (K), D96.1 (K), D97.1 (K), D98.1 (K), D99.1 (K), J12.23 (Pin_23), J12.25 (Pin_25), J12.27 (Pin_27), J13.5 (Pin_5), SW1.1, SW2.1, SW3.1, U12.16 (VSS), U12.22 (~CE1), U13.17 (GND), U13.25 (GND), U13.4 (GND)
- net RST: now also J14.17 (Pin_17), U13.33 (P33/GSR/~RST)
- net VCC: now also C28.1, C29.2, C36.1, C37.1, C38.1, J12.24 (Pin_24), J12.26 (Pin_26), J12.28 (Pin_28), R189.2, R190.2, R191.2, U12.30 (CE2), U12.32 (VCC), U13.15 (VCC), U13.26 (VCCIO), U13.35 (VCC)
- net ARAM12: now reaches U10.29 (P29/A12)
- net ARAM12: now also J14.26 (Pin_26), R154.1, U12.4 (A12)
- net ARAM13: now reaches U10.30 (P30/Z)
- net ARAM13: now also J14.28 (Pin_28), R155.1, U12.28 (A13)
- net ARAM14: now reaches U10.31 (P31/OUT0)
- net ARAM14: now also J14.21 (Pin_21), R156.1, U12.3 (A14)
- net ARAM15: now reaches U10.32 (P32/OUT1)
- net ARAM15: now also J14.23 (Pin_23), R157.1, U12.31 (A15)
- net at U10.34 (P34/GTS2/OUT2): now also U13.43 (P43/GCK1/WE)
- net at U10.36 (P36/GTS1/OUT3): now also U13.44 (P44/GCK2/OE)
- net ARAM16: now reaches U10.37 (P37/OUT4)
- net ARAM16: now also J14.25 (Pin_25), R158.1, U12.2 (A16)
- net ARAM17: now reaches U10.38 (P38/OUT5)
- net ARAM17: now also J14.27 (Pin_27), R159.1, U12.1 (A17)
- net PAGE0: now reaches U10.39 (P39/D0)
- net PAGE0: now also J14.19 (Pin_19), U13.28 (P28/AP0)
- net AIDX0 renamed ARAM0
- net ARAM0: now also J14.2 (Pin_2), R142.1, U12.12 (A0), U13.14 (P14/A0)
- net AIDX1 renamed ARAM1
- net ARAM1: now also J14.4 (Pin_4), R143.1, U12.11 (A1), U13.18 (P18/A2)
- net AIDX10 renamed ARAM10
- net ARAM10: now also J14.22 (Pin_22), R152.1, U12.23 (A10)
- net AIDX11 renamed ARAM11
- net ARAM11: now also J14.24 (Pin_24), R153.1, U12.25 (A11)
- net AIDX2 renamed ARAM2
- net ARAM2: now also J14.6 (Pin_6), R144.1, U12.10 (A2), U13.16 (P16/A1)
- net AIDX3 renamed ARAM3
- net ARAM3: now also J14.8 (Pin_8), R145.1, U12.9 (A3), U13.19 (P19/A3)
- net AIDX4 renamed ARAM4
- net ARAM4: now also J14.10 (Pin_10), R146.1, U12.8 (A4), U13.20 (P20/A4)
- net AIDX5 renamed ARAM5
- net ARAM5: now also J14.12 (Pin_12), R147.1, U12.7 (A5), U13.21 (P21/A5)
- net AIDX6 renamed ARAM6
- net ARAM6: now also J14.14 (Pin_14), R148.1, U12.6 (A6), U13.22 (P22/A6)
- net AIDX7 renamed ARAM7
- net ARAM7: now also J14.16 (Pin_16), R149.1, U12.5 (A7), U13.23 (P23/A7)
- net AIDX8 renamed ARAM8
- net ARAM8: now also J14.18 (Pin_18), R150.1, U12.27 (A8), U13.27 (P27/A8)
- net AIDX9 renamed ARAM9
- net ARAM9: now also J14.20 (Pin_20), R151.1, U12.26 (A9)
- new net: D86.2 (A), R142.2
- new net: D87.2 (A), R143.2
- new net: D88.2 (A), R144.2
- new net: D89.2 (A), R145.2
- new net: D90.2 (A), R146.2
- new net: D91.2 (A), R147.2
- new net: D92.2 (A), R148.2
- new net: D93.2 (A), R149.2
- new net: D94.2 (A), R150.2
- new net: D95.2 (A), R151.2
- new net: D96.2 (A), R152.2
- new net: D97.2 (A), R153.2
- new net: D98.2 (A), R154.2
- new net: D99.2 (A), R155.2
- new net: D100.2 (A), R156.2
- new net: D101.2 (A), R157.2
- new net: D102.2 (A), R158.2
- new net: D103.2 (A), R159.2
- new net: J12.10 (Pin_10), U13.1 (P1/GCK3/GPIO4)
- new net: J13.2 (Pin_2), U13.10 (TMS)
- new net: J13.3 (Pin_3), U13.11 (TCK)
- new net: R187.2, U13.12 (P12/D6)
- new net: R188.2, U13.13 (P13/D7)
- new net: R181.1, U13.2 (P2/D0)
- new net: J13.4 (Pin_4), U13.24 (TDO)
- new net: J12.12 (Pin_12), U13.29 (P29/GPIO5)
- new net: R182.1, U13.3 (P3/D1)
- new net: J12.14 (Pin_14), U13.30 (P30/GPIO6)
- new net: J12.16 (Pin_16), U13.31 (P31/GPIO7)
- new net: J12.18 (Pin_18), U13.32 (P32/GPIO8)
- new net: J14.29 (Pin_29), U13.34 (P34/GTS2)
- new net: J14.31 (Pin_31), U13.36 (P36/GTS1/OE_OUT)
- new net: J12.20 (Pin_20), U13.37 (P37/GPIO9)
- new net: J12.22 (Pin_22), U13.38 (P38/GPIO10)
- new net: J12.2 (Pin_2), U13.39 (P39/GPIO0)
- new net: J12.4 (Pin_4), U13.40 (P40/GPIO1)
- new net: J12.6 (Pin_6), U13.41 (P41/GPIO2)
- new net: J12.8 (Pin_8), U13.42 (P42/GPIO3)
- new net: R183.2, U13.5 (P5/D2)
- new net: R184.2, U13.6 (P6/D3)
- new net: R185.2, U13.7 (P7/D4)
- new net: R186.2, U13.8 (P8/D5)
- new net: J13.1 (Pin_1), U13.9 (TDI)
- new net: J12.1 (Pin_1), R173.1
- new net: J12.11 (Pin_11), R178.1
- new net: J12.13 (Pin_13), R179.1
- new net: J12.15 (Pin_15), R180.1
- new net: J12.3 (Pin_3), R174.1
- new net: J12.5 (Pin_5), R175.1
- new net: J12.7 (Pin_7), R176.1
- new net: J12.9 (Pin_9), R177.1
- new net: D117.2 (A), R173.2
- new net: D118.2 (A), R174.2
- new net: D119.2 (A), R175.2
- new net: D120.2 (A), R176.2
- new net: D121.2 (A), R177.2
- new net: D122.2 (A), R178.2
- new net: D123.2 (A), R179.2
- new net: D124.2 (A), R180.2
- new net: J14.30 (Pin_30), U12.29 (~WE)
- new net: J14.32 (Pin_32), U12.24 (~OE~)
- new net: R125.1, U12.13 (D0)
- new net: R126.1, U12.14 (D1)
- new net: R127.1, U12.15 (D2)
- new net: R132.2, U12.17 (D3)
- new net: R131.2, U12.18 (D4)
- new net: R130.2, U12.19 (D5)
- new net: R129.2, U12.20 (D6)
- new net: R128.2, U12.21 (D7)
- new net BTN0: C39.1, J12.17 (Pin_17), R189.1, SW1.2
- new net BTN1: C40.1, J12.19 (Pin_19), R190.1, SW2.2
- new net BTN2: C41.1, J12.21 (Pin_21), R191.1, SW3.2
Other:
- moved on the sheet: C1, C10, C11, C12, C13, C14, C15, C16, C17, C18, C19, C2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
