File: hardware/cpld-cpu.sch (KiCad schematic (older format))
At the start: 386 parts, among them J1 Acc, J10 Page, J11 PC_H, J12 Conn_02x16_Odd_Even, J13 Page, J14 Conn_02x16_Odd_Even, J2 X, J3 IR, J4 AXM, J5 Dec, J6 AR, J7 ALU, J8 Index, J9 PC_L, SW1 BTN0, SW2 BTN0, SW3 BTN0, U1 Acc, U10 RAM_Page, U11 PC_H, U12 CY62138FV30LL, U13 GPIO_RNG, U2 X, U3 IR, U4 Multiplexer, U5 Decoder, U6 AR, U7 ALU, U8 RAM_Index, U9 PC_L

Commit message: Simplify mem oe/we interface. Makes more pins available on mem_page.
Parts:
- added D125, D126: LED_Small, LEDs:LED_0805_HandSoldering, symbol Device:LED_Small
- added R192, R193: 470, Resistors_SMD:R_0805_HandSoldering, symbol Device:R_Small
- added R194, R195: 2k, Resistors_SMD:R_0805_HandSoldering, symbol Device:R_Small
- J14: value Conn_02x16_Odd_Even -> Conn_02x17_Odd_Even; symbol Connector_Generic:Conn_02x16_Odd_Even -> Connector_Generic:Conn_02x18_Odd_Even
Connections:
- net ADDR12: now also U10.29 (P29/A12); no longer U10.1 (P1/GCK3/PROG0)
- net ARAM0: now also J14.4 (Pin_4); no longer J14.2 (Pin_2)
- net ARAM1: now also J14.6 (Pin_6); no longer J14.4 (Pin_4)
- net ARAM10: now also J14.24 (Pin_24); no longer J14.22 (Pin_22)
- net ARAM11: now also J14.26 (Pin_26); no longer J14.24 (Pin_24)
- net ARAM12: now also J14.28 (Pin_28), U10.31 (P31/OUT0); no longer J14.26 (Pin_26), U10.29 (P29/A12)
- net ARAM13: now also J14.30 (Pin_30), U10.32 (P32/OUT1); no longer J14.28 (Pin_28), U10.30 (P30/Z)
- net ARAM14: now also J14.23 (Pin_23), U10.34 (P34/GTS2/OUT2); no longer J14.21 (Pin_21), U10.31 (P31/OUT0)
- net ARAM15: now also J14.25 (Pin_25), U10.36 (P36/GTS1/OUT3); no longer J14.23 (Pin_23), U10.32 (P32/OUT1)
- net ARAM16: now also J14.27 (Pin_27); no longer J14.25 (Pin_25)
- net ARAM17: now also J14.29 (Pin_29); no longer J14.27 (Pin_27)
- net ARAM2: now also J14.8 (Pin_8); no longer J14.6 (Pin_6)
- net ARAM3: now also J14.10 (Pin_10); no longer J14.8 (Pin_8)
- net ARAM4: now also J14.12 (Pin_12); no longer J14.10 (Pin_10)
- net ARAM5: now also J14.14 (Pin_14); no longer J14.12 (Pin_12)
- net ARAM6: now also J14.16 (Pin_16); no longer J14.14 (Pin_14)
- net ARAM7: now also J14.18 (Pin_18); no longer J14.16 (Pin_16)
- net ARAM8: now also J14.20 (Pin_20); no longer J14.18 (Pin_18)
- net ARAM9: now also J14.22 (Pin_22); no longer J14.20 (Pin_20)
- net D0: now also J14.3 (Pin_3); no longer J14.1 (Pin_1)
- net D1: now also J14.5 (Pin_5); no longer J14.3 (Pin_3)
- net D2: now also J14.7 (Pin_7), R133.2; no longer J14.5 (Pin_5), R133.1
- net D3: now also J14.9 (Pin_9), R134.2; no longer J14.7 (Pin_7), R134.1
- net D4: now also J14.11 (Pin_11); no longer J14.9 (Pin_9)
- net D5: now also J14.13 (Pin_13); no longer J14.11 (Pin_11)
- net D6: now also J14.15 (Pin_15), R192.1; no longer J14.13 (Pin_13)
- net D7: now also J14.17 (Pin_17), R193.1; no longer J14.15 (Pin_15)
- net GND: now also J14.36 (Pin_36), D125.1 (K), D126.1 (K)
- net PAGE0: now also J14.21 (Pin_21), U10.30 (P30/Z); no longer J14.19 (Pin_19), U10.39 (P39/D0)
- net RAM_OE: now also J14.34 (Pin_34), U12.24 (~OE~), R194.1; no longer R9.1, U10.44 (P44/GCK2), U5.2 (P2/RAM_OE)
- net RAM_WE: now also J14.31 (Pin_31), U12.29 (~WE), U13.43 (P43/GCK1/WE)
- net RST: now also J14.19 (Pin_19); no longer J14.17 (Pin_17)
- net VCC: now also J14.35 (Pin_35)
- net at U10.2 (P2/PROG1): no longer R123.1
- net at U10.3 (P3/PROG2): no longer R124.1
- net GPIO_OE: now reaches U13.44 (P44/GCK2/OE)
- net GPIO_OE: now also R9.1, U5.2 (P2/RAM_OE); no longer U10.36 (P36/GTS1/OUT3)
- net at U10.40 (P40/D1): now also R124.1
- net at U10.41 (P41/D2): now also R133.1
- net at U10.42 (P42/D3): now also R134.1
- net at U10.5 (P5/D4): now also R135.2; no longer R133.2
- net at U10.6 (P6/D5): now also R136.2; no longer R134.2
- net at U10.7 (P7/D6): now also R192.2; no longer R135.2
- net at U10.8 (P8/D7): now also R193.2; no longer R136.2
- net at U13.34 (P34/GTS2): no longer J14.29 (Pin_29)
- net DEV_OE: now reaches U13.36 (P36/GTS1/OE_OUT)
- net DEV_OE: now also J14.32 (Pin_32), R195.1; no longer J14.31 (Pin_31)
- new net: R123.1, U10.39 (P39/D0)
- new net: D126.2 (A), R195.2
- new net: D125.2 (A), R194.2
- new net CLK: J14.33 (Pin_33)
- no-connect marks 66 -> 68
Other:
- moved on the sheet: R123, R124, R133, R134, R135, R136
